File: kicad/clock.sch (KiCad schematic (older format))
At the start: 23 parts, among them SW1 SW_SPDT, SW2 SW_Push, U10 NE555, U11 74LS04, U12 74LS08, U13 74LS32, U7 74LS08, U8 NE555, U9 NE555

Commit message: design as built
Parts:
- removed U10, U8, U9: NE555, Housings_DIP:DIP-8_W7.62mm_LongPads, symbol NE555
- removed U11: 74LS04, Housings_DIP:DIP-14_W7.62mm_LongPads, symbol 74LS04
- removed U12, U7: 74LS08, Housings_DIP:DIP-14_W7.62mm_LongPads, symbol 74LS08
- removed U13: 74LS32, Housings_DIP:DIP-14_W7.62mm_LongPads, symbol 74LS32
- added C901: 100n, Capacitors_THT:C_Disc_D6_P5, symbol C
- added C902, C903: 10n, Capacitors_THT:C_Disc_D6_P5, symbol C
- added R904: 1M, Resistors_THT:Resistor_Horizontal_RM7mm, symbol R
- added R906: 1K, Resistors_THT:Resistor_Horizontal_RM7mm, symbol R
- added R907: 100K, Resistors_THT:Resistor_Horizontal_RM7mm, symbol R
- added U901, U902: NE556, symbol NE556
- added U903: 74LS04, Housings_DIP:DIP-14_W7.62mm_LongPads, symbol 74LS04
- added U904: 74LS10, Housings_DIP:DIP-14_W7.62mm_LongPads, symbol 74LS10
- C904: renamed from C2; value 0.1uF -> 10n
- C905: renamed from C1; value 0.1uF -> 10n
- C906: renamed from C3; value 0.1uF -> 10n
- C907: renamed from C5; value 0.1u -> 330n
- R903: renamed from R3; value 1K -> 10K
- R911: renamed from R8; value 220 -> 1K
- SW901: renamed from SW1; value SW_SPDT -> SW_Select; footprint Buttons_Switches_THT:SW_Micro_SPST -> Buttons_Switches_THT:SW_PUSH_x2
- SW902: renamed from SW2; value SW_Push -> SW_Manual
- renumbered C4 to C908, D1 to D901, R1 to R901, R2 to R902, R5 to R905, R7 to R908, R6 to R909, R4 to R910
Connections:
- net labels added: CLK2, DCLK, ZERO, ~ZERO
- net labels removed: ~CLK
- wire segments 64 -> 95
- no-connect marks 1 -> 2
Other:
- moved on the sheet: C904, C905, C906, C907, C908, D901, R901, R902, R903, R905, R908, R909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
