File: kicad/clock.sch (KiCad schematic (older format))
At the start: 22 parts, among them SW1 SW_SPDT, SW2 SW_Push, U30 NE555, U31 NE555, U32 74LS04, U33 74LS08, U34 74LS32, U6 NE555

Commit message: bugfixed design
Parts:
- renumbered C5 to C1, C1 to C2, C6 to C3, C2 to C4, C7 to C5, R22 to R1, R23 to R2, R24 to R3, R1 to R4, R25 to R5, R2 to R6, R4 to R7, R3 to R8, U31 to U10, U32 to U11, U33 to U12, U34 to U13, U33 to U7, U6 to U8, U30 to U9
Changed lines of the file:
@@
 LIBS:valves
 LIBS:switches
-LIBS:74xxx
-LIBS:28c16
 LIBS:sap-be-cache
-EELAYER 24 0
+EELAYER 25 0
 EELAYER END
 $Descr A4 11693 8268
@@
 $EndDescr
 $Comp
-L NE555 U6
+L NE555 U8
 U 1 1 591AA275
 P 2700 1250
-F 0 "U6" H 2300 1600 50  0000 L CNN
+F 0 "U8" H 2300 1600 50  0000 L CNN
 F 1 "NE555" H 2300 900 50  0000 L CNN
 F 2 "Housings_DIP:DIP-8_W7.62mm_LongPads" H 2700 1250 50  0001 C CNN
@@
 $EndComp
 $Comp
-L R_Variable R2
+L R_Variable R6
 U 1 1 591AB200
 P 3750 1450
-F 0 "R2" V 3850 1350 50  0000 L CNN
+F 0 "R6" V 3850 1350 50  0000 L CNN
 F 1 "1M" V 3650 1400 50  0000 L CNN
 F 2 "Potentiometers:Potentiometer_Alps-RK16-single" V 3680 1450 50  0001 C CNN
@@
 $EndComp
 $Comp
-L R R1
+L R R4
 U 1 1 591AB2B7
 P 3400 1450
-F 0 "R1" V 3480 1450 50  0000 C CNN
+F 0 "R4" V 3480 1450 50  0000 C CNN
 F 1 "1K" V 3400 1450 50  0000 C CNN
 F 2 "Resistors_THT:Resistor_Horizontal_RM7mm" V 3330 1450 50  0001 C CNN
@@
 $EndComp
 $Comp
-L GND #PWR012
+L GND #PWR17
 U 1 1 591AB594
 P 3250 2200
-F 0 "#PWR012" H 3250 1950 50  0001 C CNN
+F 0 "#PWR17" H 3250 1950 50  0001 C CNN
 F 1 "GND" H 3250 2050 50  0000 C CNN
 F 2 "" H 3250 2200 50  0000 C CNN
@@
 $EndComp
 $Comp
-L CP C2
+L CP C4
 U 1 1 591AB5AE
 P 3250 2000
-F 0 "C2" H 3275 2100 50  0000 L CNN
+F 0 "C4" H 3275 2100 50  0000 L CNN
 F 1 "1uF" H 3275 1900 50  0000 L CNN
 F 2 "Capacitors_THT:C_Radial_D5_L11_P2" H 3288 1850 50  0001 C CNN
@@
 $EndComp
 $Comp
-L VCC #PWR013
+L VCC #PWR21
 U 1 1 591AB7DD
 P 4400 1450
-F 0 "#PWR013" H 4400 1300 50  0001 C CNN
+F 0 "#PWR21" H 4400 1300 50  0001 C CNN
 F 1 "VCC" H 4400 1600 50  0000 C CNN
 F 2 "" H 4400 1450 50  0000 C CNN
@@
 $EndComp
 $Comp
-L R R4
+L R R7
 U 1 1 591AB86C
 P 4150 1450
-F 0 "R4" V 4230 1450 50  0000 C CNN
+F 0 "R7" V 4230 1450 50  0000 C CNN
 F 1 "1K" V 4150 1450 50  0000 C CNN
 F 2 "Resistors_THT:Resistor_Horizontal_RM7mm" V 4080 1450 50  0001 C CNN
@@
 $EndComp
 $Comp
-L R R3
+L R R8
 U 1 1 591ABE42
 P 9750 4350
-F 0 "R3" V 9830 4350 50  0000 C CNN
+F 0 "R8" V 9830 4350 50  0000 C CNN
 F 1 "220" V 9750 4350 50  0000 C CNN
 F 2 "Resistors_THT:Resistor_Horizontal_RM7mm" V 9680 4350 50  0001 C CNN
@@
 	9750 4100 9750 4200
 $Comp
-L GND #PWR014
+L GND #PWR22
 U 1 1 591ABF50
 P 9750 4550
-F 0 "#PWR014" H 9750 4300 50  0001 C CNN
+F 0 "#PWR22" H 9750 4300 50  0001 C CNN
 F 1 "GND" H 9750 4400 50  0000 C CNN
 F 2 "" H 9750 4550 50  0000 C CNN
@@
 	3250 2200 3250 2150
 $Comp
-L GND #PWR015
+L GND #PWR12
 U 1 1 591AC3CA
 P 1650 1250
-F 0 "#PWR015" H 1650 1000 50  0001 C CNN
+F 0 "#PWR12" H 1650 1000 50  0001 C CNN
 F 1 "GND" H 1650 1100 50  0000 C CNN
 F 2 "" H 1650 1250 50  0000 C CNN
@@
 $EndComp
 $Comp
-L C C1
+L C C2
 U 1 1 591AC401
 P 1900 1250
-F 0 "C1" H 1925 1350 50  0000 L CNN
+F 0 "C2" H 1925 1350 50  0000 L CNN
 F 1 "0.1uF" H 1925 1150 50  0000 L CNN
 F 2 "Capacitors_THT:C_Disc_D6_P5" H 1938 1100 50  0001 C CNN
@@
 	1750 1250 1650 1250
 $Comp
-L VCC #PWR016
+L VCC #PWR16
 U 1 1 590D1C81
 P 2150 1450
-F 0 "#PWR016" H 2150 1300 50  0001 C CNN
+F 0 "#PWR16" H 2150 1300 50  0001 C CNN
 F 1 "VCC" H 2150 1600 50  0000 C CNN
 F 2 "" H 2150 1450 50  0000 C CNN
@@
 ~CLK
 $Comp
-L NE555 U30
+L NE555 U9
 U 1 1 59264260
 P 2700 3400
-F 0 "U30" H 2300 3750 50  0000 L CNN
+F 0 "U9" H 2300 3750 50  0000 L CNN
 F 1 "NE555" H 2300 3050 50  0000 L CNN
 F 2 "Housings_DIP:DIP-8_W7.62mm_LongPads" H 2700 3400 50  0001 C CNN
@@
 $EndComp
 $Comp
-L NE555 U31
+L NE555 U10
 U 1 1 59264481
 P 2700 5350
-F 0 "U31" H 2300 5700 50  0000 L CNN
+F 0 "U10" H 2300 5700 50  0000 L CNN
 F 1 "NE555" H 2300 5000 50  0000 L CNN
 F 2 "Housings_DIP:DIP-8_W7.62mm_LongPads" H 2700 5350 50  0001 C CNN
@@
 $EndComp
 $Comp
-L GND #PWR017
+L GND #PWR11
 U 1 1 59124B4A
 P 1400 3400
-F 0 "#PWR017" H 1400 3150 50  0001 C CNN
+F 0 "#PWR11" H 1400 3150 50  0001 C CNN
 F 1 "GND" H 1400 3250 50  0000 C CNN
 F 2 "" H 1400 3400 50  0000 C CNN
@@
 $EndComp
 $Comp
-L R R24
+L R R3
 U 1 1 59124B76
 P 2100 3000
-F 0 "R24" V 2180 3000 50  0000 C CNN
+F 0 "R3" V 2180 3000 50  0000 C CNN
 F 1 "1K" V 2100 3000 50  0000 C CNN
 F 2 "Resistors_THT:Resistor_Horizontal_RM7mm" V 2030 3000 50  0001 C CNN
@@
 $EndComp
 $Comp
-L VCC #PWR018
+L VCC #PWR14
 U 1 1 59124C74
 P 2100 2800
-F 0 "#PWR018" H 2100 2650 50  0001 C CNN
+F 0 "#PWR14" H 2100 2650 50  0001 C CNN
 F 1 "VCC" H 2100 2950 50  0000 C CNN
 F 2 "" H 2100 2800 50  0000 C CNN
@@
 	3350 3400 3200 3400
 $Comp
-L R R25
+L R R5
 U 1 1 59124FED
 P 3500 3400
-F 0 "R25" V 3580 3400 50  0000 C CNN
+F 0 "R5" V 3580 3400 50  0000 C CNN
 F 1 "1M" V 3500 3400 50  0000 C CNN
 F 2 "Resistors_THT:Resistor_Horizontal_RM7mm" V 3430 3400 50  0001 C CNN
@@
 $EndComp
 $Comp
-L C C7
+L C C5
 U 1 1 59125085
 P 3350 3750
-F 0 "C7" H 3375 3850 50  0000 L CNN
+F 0 "C5" H 3375 3850 50  0000 L CNN
 F 1 "0.1u" H 3375 3650 50  0000 L CNN
 F 2 "Capacitors_THT:C_Disc_D6_P5" H 3388 3600 50  0001 C CNN
@@
 $EndComp
 $Comp
-L GND #PWR019
+L GND #PWR19
 U 1 1 591250DE
 P 3350 4000
-F 0 "#PWR019" H 3350 3750 50  0001 C CNN
+F 0 "#PWR19" H 3350 3750 50  0001 C CNN
 F 1 "GND" H 3350 3850 50  0000 C CNN
 F 2 "" H 3350 4000 50  0000 C CNN
@@
 	2100 2800 2100 2850
 $Comp
-L C C5
+L C C1
 U 1 1 5912559C
 P 1800 3400
-F 0 "C5" H 1825 3500 50  0000 L CNN
+F 0 "C1" H 1825 3500 50  0000 L CNN
 F 1 "0.1uF" H 1825 3300 50  0000 L CNN
 F 2 "Capacitors_THT:C_Disc_D6_P5" H 1838 3250 50  0001 C CNN
@@
 	2200 3400 1950 3400
 $Comp
-L VCC #PWR020
+L VCC #PWR15
 U 1 1 59126100
 P 2100 3600
-F 0 "#PWR020" H 2100 3450 50  0001 C CNN
+F 0 "#PWR15" H 2100 3450 50  0001 C CNN
 F 1 "VCC" H 2100 3750 50  0000 C CNN
 F 2 "" H 2100 3600 50  0000 C CNN
@@
 	2200 1450 2150 1450
 $Comp
-L VCC #PWR021
+L VCC #PWR20
 U 1 1 59126A90
 P 3750 3400
-F 0 "#PWR021" H 3750 3250 50  0001 C CNN
+F 0 "#PWR20" H 3750 3250 50  0001 C CNN
 F 1 "VCC" H 3750 3550 50  0000 C CNN
 F 2 "" H 3750 3400 50  0000 C CNN
@@
 	3650 3400 3750 3400
 $Comp
-L GND #PWR022
+L GND #PWR18
 U 1 1 59128FED
 P 3300 5550
-F 0 "#PWR022" H 3300 5300 50  0001 C CNN
+F 0 "#PWR18" H 3300 5300 50  0001 C CNN
 F 1 "GND" H 3300 5400 50  0000 C CNN
 F 2 "" H 3300 5550 50  0000 C CNN
@@
 	3200 5550 3300 5550
 $Comp
-L R R23
+L R R2
 U 1 1 59129512
 P 1150 4950
-F 0 "R23" V 1230 4950 50  0000 C CNN
+F 0 "R2" V 1230 4950 50  0000 C CNN
 F 1 "1K" V 1150 4950 50  0000 C CNN
 F 2 "Resistors_THT:Resistor_Horizontal_RM7mm" V 1080 4950 50  0001 C CNN
@@
 $EndComp
 $Comp
-L R R22
+L R R1
 U 1 1 59129597
 P 950 4950
-F 0 "R22" V 1030 4950 50  0000 C CNN
+F 0 "R1" V 1030 4950 50  0000 C CNN
 F 1 "1K" V 950 4950 50  0000 C CNN
 F 2 "Resistors_THT:Resistor_Horizontal_RM7mm" V 880 4950 50  0001 C CNN
@@
 $EndComp
 $Comp
-L VCC #PWR023
+L VCC #PWR10
 U 1 1 5912968A
 P 1050 4750
-F 0 "#PWR023" H 1050 4600 50  0001 C CNN
+F 0 "#PWR10" H 1050 4600 50  0001 C CNN
 F 1 "VCC" H 1050 4900 50  0000 C CNN
 F 2 "" H 1050 4750 50  0000 C CNN
@@
 $EndComp
 $Comp
-L GND #PWR024
+L GND #PWR13
 U 1 1 5912A8EB
 P 1700 5500
-F 0 "#PWR024" H 1700 5250 50  0001 C CNN
+F 0 "#PWR13" H 1700 5250 50  0001 C CNN
 F 1 "GND" H 1700 5350 50  0000 C CNN
 F 2 "" H 1700 5500 50  0000 C CNN
@@
 $EndComp
 $Comp
-L C C6
+L C C3
 U 1 1 5912AC95
 P 1950 5350
-F 0 "C6" H 1975 5450 50  0000 L CNN
+F 0 "C3" H 1975 5450 50  0000 L CNN
 F 1 "0.1uF" H 1975 5250 50  0000 L CNN
 F 2 "Capacitors_THT:C_Disc_D6_P5" H 1988 5200 50  0001 C CNN
@@
 ASTABLE
 $Comp
-L 74LS04 U32
+L 74LS04 U11
 U 1 1 591302C9
 P 5300 3650
-F 0 "U32" H 5495 3765 50  0000 C CNN
+F 0 "U11" H 5495 3765 50  0000 C CNN
 F 1 "74LS04" H 5490 3525 50  0000 C CNN
 F 2 "Housings_DIP:DIP-14_W7.62mm_LongPads" H 5300 3650 50  0001 C CNN
@@
 $EndComp
 $Comp
-L 74LS04 U32
+L 74LS04 U11
 U 3 1 5913032A
 P 10200 3400
-F 0 "U32" H 10395 3515 50  0000 C CNN
+F 0 "U11" H 10395 3515 50  0000 C CNN
 F 1 "74LS04" H 10390 3275 50  0000 C CNN
 F 2 "Housings_DIP:DIP-14_W7.62mm_LongPads" H 10200 3400 50  0001 C CNN
@@
 $EndComp
 $Comp
-L 74LS04 U32
+L 74LS04 U11
 U 2 1 59130373
 P 5300 4250
-F 0 "U32" H 5495 4365 50  0000 C CNN
+F 0 "U11" H 5495 4365 50  0000 C CNN
 F 1 "74LS04" H 5490 4125 50  0000 C CNN
 F 2 "Housings_DIP:DIP-14_W7.62mm_LongPads" H 5300 4250 50  0001 C CNN
@@
 $EndComp
 $Comp
-L 74LS08 U33
-U 3 1 591303CC
+L 74LS08 U12
+U 2 1 591303CC
 P 9050 3600
-F 0 "U33" H 9050 3650 50  0000 C CNN
+F 0 "U12" H 9050 3650 50  0000 C CNN
 F 1 "74LS08" H 9050 3550 50  0000 C CNN
 F 2 "Housings_DIP:DIP-14_W7.62mm_LongPads" H 9050 3600 50  0001 C CNN
 F 3 "" H 9050 3600 50  0000 C CNN
-	3    9050 3600
-	1    0    0    -1
-$EndComp
-$Comp
-L 74LS08 U33
-U 1 1 5913048F
+	2    9050 3600
+	1    0    0    -1
+$EndComp
+$Comp
+L 74LS08 U7
+U 4 1 5913048F
 P 6450 3250
-F 0 "U33" H 6450 3300 50  0000 C CNN
+F 0 "U7" H 6450 3300 50  0000 C CNN
 F 1 "74LS08" H 6450 3200 50  0000 C CNN
 F 2 "Housings_DIP:DIP-14_W7.62mm_LongPads" H 6450 3250 50  0001 C CNN
 F 3 "" H 6450 3250 50  0000 C CNN
-	1    6450 3250
-	1    0    0    -1
-$EndComp
-$Comp
-L 74LS08 U33
-U 2 1 591304E2
+	4    6450 3250
+	1    0    0    -1
+$EndComp
+$Comp
+L 74LS08 U12
+U 1 1 591304E2
 P 6450 3750
-F 0 "U33" H 6450 3800 50  0000 C CNN
+F 0 "U12" H 6450 3800 50  0000 C CNN
 F 1 "74LS08" H 6450 3700 50  0000 C CNN
 F 2 "Housings_DIP:DIP-14_W7.62mm_LongPads" H 6450 3750 50  0001 C CNN
 F 3 "" H 6450 3750 50  0000 C CNN
-	2    6450 3750
-	1    0    0    -1
-$EndComp
-$Comp
-L 74LS32 U34
+	1    6450 3750
+	1    0    0    -1
+$EndComp
+$Comp
+L 74LS32 U13
 U 1 1 5913052F
 P 7750 3500
-F 0 "U34" H 7750 3550 50  0000 C CNN
+F 0 "U13" H 7750 3550 50  0000 C CNN
 F 1 "74LS32" H 7750 3450 50  0000 C CNN
 F 2 "Housings_DIP:DIP-14_W7.62mm_LongPads" H 7750 3500 50  0001 C CNN

Commit message: Update bugfix version to use updated kicad libraries
Parts:
- removed C1, C2, C3: 0.1uF, Capacitors_THT:C_Disc_D6_P5, symbol C
- removed C4: 1uF, Capacitors_THT:C_Radial_D5_L11_P2, symbol CP
- removed C5: 0.1u, Capacitors_THT:C_Disc_D6_P5, symbol C
- removed D1: LED, LEDs:LED-5MM, symbol LED
- removed R1, R2, R3, R4, R7: 1K, Resistors_THT:Resistor_Horizontal_RM7mm, symbol R
- removed R5: 1M, Resistors_THT:Resistor_Horizontal_RM7mm, symbol R
- removed R6: 1M, Potentiometers:Potentiometer_Alps-RK16-single, symbol R_Variable
- removed R8: 220, Resistors_THT:Resistor_Horizontal_RM7mm, symbol R
- removed SW1: SW_SPDT, Buttons_Switches_THT:SW_Micro_SPST, symbol SW_SPDT
- removed SW2: SW_Push, Buttons_Switches_THT:SW_PUSH_6mm_h9.5mm, symbol SW_Push
- removed U10, U8, U9: NE555, Housings_DIP:DIP-8_W7.62mm_LongPads, symbol NE555
- removed U11: 74LS04, Housings_DIP:DIP-14_W7.62mm_LongPads, symbol 74LS04
- removed U12, U7: 74LS08, Housings_DIP:DIP-14_W7.62mm_LongPads, symbol 74LS08
- removed U13: 74LS32, Housings_DIP:DIP-14_W7.62mm_LongPads, symbol 74LS32
- added C1, C2, C3, C5: 0.1uF, symbol Device:C
- added C4: 1uF, symbol Device:CP
- added D1: LED, symbol Device:LED
- added R1, R2, R3, R4, R7: 1K, symbol Device:R
- added R5: 1M, symbol Device:R
- added R6: 1M, symbol Device:RTRIM
- added R8: 220, symbol Device:R
- added SW1: source select, symbol Switch:SW_SPDT
- added SW2: Manual, symbol Switch:SW_Push
- added U10: 74LS32, symbol 74xx:74LS32
- added U11, U12, U13: LM555, symbol Timer:LM555
- added U8: 74LS04, symbol 74xx:74LS04
- added U9: 74LS08, symbol 74xx:74LS08
Connections:
- wire segments 64 -> 81
