File: kicad/clock.sch (KiCad schematic (older format))
At the start: 22 parts, among them SW1 SW_SPDT, SW2 SW_Push, U30 NE555, U31 NE555, U32 74LS04, U33 74LS08, U34 74LS32, U6 NE555

Commit message: Update to current kicad libraries
Parts:
- removed C1, C5, C6: 0.1uF, Capacitors_THT:C_Disc_D6_P5, symbol C
- removed C2: 1uF, Capacitors_THT:C_Radial_D5_L11_P2, symbol CP
- removed C7: 0.1u, Capacitors_THT:C_Disc_D6_P5, symbol C
- removed D1: LED, LEDs:LED-5MM, symbol LED
- removed R1, R22, R23, R24, R4: 1K, Resistors_THT:Resistor_Horizontal_RM7mm, symbol R
- removed R2: 1M, Potentiometers:Potentiometer_Alps-RK16-single, symbol R_Variable
- removed R25: 1M, Resistors_THT:Resistor_Horizontal_RM7mm, symbol R
- removed R3: 220, Resistors_THT:Resistor_Horizontal_RM7mm, symbol R
- removed SW1: SW_SPDT, Buttons_Switches_THT:SW_Micro_SPST, symbol SW_SPDT
- removed SW2: SW_Push, Buttons_Switches_THT:SW_PUSH_6mm_h9.5mm, symbol SW_Push
- removed U30, U31, U6: NE555, Housings_DIP:DIP-8_W7.62mm_LongPads, symbol NE555
- removed U32: 74LS04, Housings_DIP:DIP-14_W7.62mm_LongPads, symbol 74LS04
- removed U33: 74LS08, Housings_DIP:DIP-14_W7.62mm_LongPads, symbol 74LS08
- removed U34: 74LS32, Housings_DIP:DIP-14_W7.62mm_LongPads, symbol 74LS32
- added C1, C2, C3, C5: 0.1uF, symbol Device:C
- added C4: 1uF, symbol Device:CP
- added D1: LED, symbol Device:LED
- added R1, R2, R3, R4, R7: 1K, symbol Device:R
- added R5: 1M, symbol Device:R
- added R6: 1M, symbol Device:RTRIM
- added R8: 220, symbol Device:R
- added SW1: source select, symbol Switch:SW_SPDT
- added SW2: Manual, symbol Switch:SW_Push
- added U10: 74LS32, symbol 74xx:74LS32
- added U11, U12, U13: LM555, symbol Timer:LM555
- added U8: 74LS04, symbol 74xx:74LS04
- added U9: 74LS08, symbol 74xx:74LS08
Connections:
- wire segments 64 -> 81

Commit message: update bus names and improve sheet text
Parts:
- added U7: 74LS04, symbol 74xx:74LS04
- added U8: 74LS08, symbol 74xx:74LS08
- added U9: 74LS32, symbol 74xx:74LS32
- renumbered C3 to C2, C2 to C3, U11 to U1, U13 to U2, U12 to U3, U8 to U4, U9 to U5, U10 to U6
