File: kicad/sap-be.sch (KiCad schematic (older format))
At the start: 0 parts

Commit message: design as built
Connections:
- net labels added: DCLK, ZERO, i[0..7], ~ZERO
- net labels removed: ZRO
- wire segments 95 -> 99
