File: kicad/sap-be.sch (KiCad schematic (older format))
At the start: 0 parts

Commit message: Update to current kicad libraries
Connections:
- net labels added: PGM, a[0..3], ra[0..7], rb[0..7]
- net labels removed: CLR, a[0..7], b[0..7]
- wire segments 95 -> 92
