File: kicad/register.sch (KiCad schematic (older format))
At the start: 11 parts, among them U14 74LS173, U15 74LS173, U16 74LS245

Commit message: design as built
Parts:
- renumbered D2 to D301, D3 to D302, D4 to D303, D5 to D304, D6 to D305, D7 to D306, D8 to D307, D9 to D308, U14 to U301, U15 to U302, U16 to U303

Commit message: Update to current kicad version
Parts:
- removed D301, D302, D303, D304, D305, D306, D307, D308: LED, LEDs:LED-5MM, symbol LED
- removed U301, U302: 74LS173, Housings_DIP:DIP-16_W7.62mm_LongPads, symbol 74LS173
- removed U303: 74LS245, Housings_DIP:DIP-20_W7.62mm_LongPads, symbol 74LS245
- added BAR2: HDSP-4830_2, Display:HDSP-4830, symbol LED:HDSP-4830_2
- added RN3: 1K, Resistor_THT:R_Array_SIP9, symbol Device:R_Network08
- added U3: 74LS245, symbol 74xx:74LS245
- added U4, U5: 74LS173, symbol 74xx:74LS173
Connections:
- net labels removed: ~RENABLE
- wire segments 73 -> 66
- no-connect marks 0 -> 4
