File: kicad/control.sch (KiCad schematic (older format))
At the start: 16 parts, among them SW7 SW_Push, U24 74LS161, U25 28C16, U26 74LS138, U27 28C16, U42 74LS00, U45 74LS00

Commit message: bugfixed design
Parts:
- renumbered D59 to D36, D60 to D37, D61 to D38, D62 to D39, D63 to D40, D64 to D41, D65 to D42, D66 to D43, R29 to R23, SW7 to SW5, U42 to U33, U24 to U37, U25 to U38, U26 to U39, U42 to U40, U45 to U40, U27 to U41
Changed lines of the file:
@@
 LIBS:valves
 LIBS:switches
-LIBS:74xxx
-LIBS:28c16
 LIBS:sap-be-cache
-EELAYER 24 0
+EELAYER 25 0
 EELAYER END
 $Descr A4 11693 8268
@@
 ~CLK
 $Comp
-L 74LS161 U24
+L 74LS161 U37
 U 1 1 591DFF5B
 P 2350 3100
-F 0 "U24" H 2400 3200 50  0000 C CNN
+F 0 "U37" H 2400 3200 50  0000 C CNN
 F 1 "74LS161" H 2450 2900 50  0000 C CNN
 F 2 "Housings_DIP:DIP-16_W7.62mm_LongPads" H 2350 3100 50  0001 C CNN
@@
 $EndComp
 $Comp
-L VCC #PWR056
+L VCC #PWR55
 U 1 1 591E000C
 P 1550 3100
-F 0 "#PWR056" H 1550 2950 50  0001 C CNN
+F 0 "#PWR55" H 1550 2950 50  0001 C CNN
 F 1 "VCC" H 1550 3250 50  0000 C CNN
 F 2 "" H 1550 3100 50  0000 C CNN
@@
 i[0..7]
 $Comp
-L 74LS138 U26
+L 74LS138 U39
 U 1 1 591E008D
 P 4100 2950
-F 0 "U26" H 4200 3450 50  0000 C CNN
+F 0 "U39" H 4200 3450 50  0000 C CNN
 F 1 "74LS138" H 4250 2401 50  0000 C CNN
 F 2 "Housings_DIP:DIP-16_W7.62mm_LongPads" H 4100 2950 50  0001 C CNN
@@
 $EndComp
 $Comp
-L GND #PWR057
+L GND #PWR62
 U 1 1 591E00E0
 P 3400 3300
-F 0 "#PWR057" H 3400 3050 50  0001 C CNN
+F 0 "#PWR62" H 3400 3050 50  0001 C CNN
 F 1 "GND" H 3400 3150 50  0000 C CNN
 F 2 "" H 3400 3300 50  0000 C CNN
@@
 $EndComp
 $Comp
-L VCC #PWR058
+L VCC #PWR61
 U 1 1 591E013C
 P 3400 3100
-F 0 "#PWR058" H 3400 2950 50  0001 C CNN
+F 0 "#PWR61" H 3400 2950 50  0001 C CNN
 F 1 "VCC" H 3400 3250 50  0000 C CNN
 F 2 "" H 3400 3100 50  0000 C CNN
@@
 J
 $Comp
-L 28C16 U25
+L 28C16 U38
 U 1 1 59257375
 P 3650 5250
-F 0 "U25" H 3850 6250 50  0000 C CNN
+F 0 "U38" H 3850 6250 50  0000 C CNN
 F 1 "28C16" H 3950 4250 50  0000 C CNN
 F 2 "Housings_DIP:DIP-24_W15.24mm_LongPads" H 3650 5250 50  0001 C CNN
@@
 $EndComp
 $Comp
-L 28C16 U27
+L 28C16 U41
 U 1 1 59257567
 P 7500 5250
-F 0 "U27" H 7700 6250 50  0000 C CNN
+F 0 "U41" H 7700 6250 50  0000 C CNN
 F 1 "28C16" H 7800 4250 50  0000 C CNN
 F 2 "Housings_DIP:DIP-24_W15.24mm_LongPads" H 7500 5250 50  0001 C CNN
@@
 CF
 $Comp
-L GND #PWR059
+L GND #PWR60
 U 1 1 59258439
 P 2700 6200
-F 0 "#PWR059" H 2700 5950 50  0001 C CNN
+F 0 "#PWR60" H 2700 5950 50  0001 C CNN
 F 1 "GND" H 2700 6050 50  0000 C CNN
 F 2 "" H 2700 6200 50  0000 C CNN
@@
 $EndComp
 $Comp
-L VCC #PWR060
+L VCC #PWR59
 U 1 1 592584B3
 P 2700 5900
-F 0 "#PWR060" H 2700 5750 50  0001 C CNN
+F 0 "#PWR59" H 2700 5750 50  0001 C CNN
 F 1 "VCC" H 2700 6050 50  0000 C CNN
 F 2 "" H 2700 5900 50  0000 C CNN
@@
 $EndComp
 $Comp
-L VCC #PWR061
+L VCC #PWR66
 U 1 1 5925973D
 P 6550 5900
-F 0 "#PWR061" H 6550 5750 50  0001 C CNN
+F 0 "#PWR66" H 6550 5750 50  0001 C CNN
 F 1 "VCC" H 6550 6050 50  0000 C CNN
 F 2 "" H 6550 5900 50  0000 C CNN
@@
 $EndComp
 $Comp
-L GND #PWR062
+L GND #PWR67
 U 1 1 59259759
 P 6550 6200
-F 0 "#PWR062" H 6550 5950 50  0001 C CNN
+F 0 "#PWR67" H 6550 5950 50  0001 C CNN
 F 1 "GND" H 6550 6050 50  0000 C CNN
 F 2 "" H 6550 6200 50  0000 C CNN
@@
 s2
 $Comp
-L GND #PWR063
+L GND #PWR58
 U 1 1 59239DA4
 P 2700 5450
-F 0 "#PWR063" H 2700 5200 50  0001 C CNN
+F 0 "#PWR58" H 2700 5200 50  0001 C CNN
 F 1 "GND" H 2700 5300 50  0000 C CNN
 F 2 "" H 2700 5450 50  0000 C CNN
@@
 i7
 $Comp
-L GND #PWR064
+L GND #PWR65
 U 1 1 5923A353
 P 6550 5450
-F 0 "#PWR064" H 6550 5200 50  0001 C CNN
+F 0 "#PWR65" H 6550 5200 50  0001 C CNN
 F 1 "GND" H 6550 5300 50  0000 C CNN
 F 2 "" H 6550 5450 50  0000 C CNN
@@
 NoConn ~ 4900 3200
 $Comp
-L LED D62
+L LED D39
 U 1 1 5923AFFE
 P 7300 2850
-F 0 "D62" H 7300 2950 50  0000 C CNN
+F 0 "D39" H 7300 2950 50  0000 C CNN
 F 1 "LED" H 7300 2750 50  0000 C CNN
 F 2 "" H 7300 2850 50  0000 C CNN
@@
 $EndComp
 $Comp
-L LED D63
+L LED D40
 U 1 1 5923B080
 P 7600 2850
-F 0 "D63" H 7600 2950 50  0000 C CNN
+F 0 "D40" H 7600 2950 50  0000 C CNN
 F 1 "LED" H 7600 2750 50  0000 C CNN
 F 2 "" H 7600 2850 50  0000 C CNN
@@
 $EndComp
 $Comp
-L LED D64
+L LED D41
 U 1 1 5923B0BE
 P 7900 2850
-F 0 "D64" H 7900 2950 50  0000 C CNN
+F 0 "D41" H 7900 2950 50  0000 C CNN
 F 1 "LED" H 7900 2750 50  0000 C CNN
 F 2 "" H 7900 2850 50  0000 C CNN
@@
 $EndComp
 $Comp
-L LED D65
+L LED D42
 U 1 1 5923B0EF
 P 8200 2850
-F 0 "D65" H 8200 2950 50  0000 C CNN
+F 0 "D42" H 8200 2950 50  0000 C CNN
 F 1 "LED" H 8200 2750 50  0000 C CNN
 F 2 "" H 8200 2850 50  0000 C CNN
@@
 $EndComp
 $Comp
-L LED D66
+L LED D43
 U 1 1 5923B11F
 P 8500 2850
-F 0 "D66" H 8500 2950 50  0000 C CNN
+F 0 "D43" H 8500 2950 50  0000 C CNN
 F 1 "LED" H 8500 2750 50  0000 C CNN
 F 2 "" H 8500 2850 50  0000 C CNN
@@
 ~t4
 $Comp
-L GND #PWR065
+L GND #PWR68
 U 1 1 5923B94B
 P 7900 3200
-F 0 "#PWR065" H 7900 2950 50  0001 C CNN
+F 0 "#PWR68" H 7900 2950 50  0001 C CNN
 F 1 "GND" H 7900 3050 50  0000 C CNN
 F 2 "" H 7900 3200 50  0000 C CNN
@@
 $EndComp
 $Comp
-L LED D59
+L LED D36
 U 1 1 5923BD6A
 P 6150 2850
-F 0 "D59" H 6150 2950 50  0000 C CNN
+F 0 "D36" H 6150 2950 50  0000 C CNN
 F 1 "LED" H 6150 2750 50  0000 C CNN
 F 2 "" H 6150 2850 50  0000 C CNN
@@
 $EndComp
 $Comp
-L LED D60
+L LED D37
 U 1 1 5923BD70
 P 6450 2850
-F 0 "D60" H 6450 2950 50  0000 C CNN
+F 0 "D37" H 6450 2950 50  0000 C CNN
 F 1 "LED" H 6450 2750 50  0000 C CNN
 F 2 "" H 6450 2850 50  0000 C CNN
@@
 $EndComp
 $Comp
-L LED D61
+L LED D38
 U 1 1 5923BD76
 P 6750 2850
-F 0 "D61" H 6750 2950 50  0000 C CNN
+F 0 "D38" H 6750 2950 50  0000 C CNN
 F 1 "LED" H 6750 2750 50  0000 C CNN
 F 2 "" H 6750 2850 50  0000 C CNN
@@
 s2
 $Comp
-L GND #PWR066
+L GND #PWR64
 U 1 1 5923BD87
 P 6450 3200
-F 0 "#PWR066" H 6450 2950 50  0001 C CNN
+F 0 "#PWR64" H 6450 2950 50  0001 C CNN
 F 1 "GND" H 6450 3050 50  0000 C CNN
 F 2 "" H 6450 3200 50  0000 C CNN
@@
 $EndComp
 $Comp
-L 74LS00 U42
-U 2 1 59303A6C
+L 74LS00 U33
+U 4 1 59303A6C
 P 2800 1250
-F 0 "U42" H 2800 1300 50  0000 C CNN
+F 0 "U33" H 2800 1300 50  0000 C CNN
 F 1 "74LS00" H 2800 1150 50  0000 C CNN
 F 2 "" H 2800 1250 50  0000 C CNN
 F 3 "" H 2800 1250 50  0000 C CNN
-	2    2800 1250
-	1    0    0    -1
-$EndComp
-$Comp
-L 74LS00 U42
-U 3 1 59303AFF
+	4    2800 1250
+	1    0    0    -1
+$EndComp
+$Comp
+L 74LS00 U40
+U 1 1 59303AFF
 P 4500 1250
-F 0 "U42" H 4500 1300 50  0000 C CNN
+F 0 "U40" H 4500 1300 50  0000 C CNN
 F 1 "74LS00" H 4500 1150 50  0000 C CNN
 F 2 "" H 4500 1250 50  0000 C CNN
 F 3 "" H 4500 1250 50  0000 C CNN
-	3    4500 1250
-	1    0    0    -1
-$EndComp
-$Comp
-L 74LS00 U42
-U 4 1 59303B52
+	1    4500 1250
+	1    0    0    -1
+$EndComp
+$Comp
+L 74LS00 U40
+U 2 1 59303B52
 P 4500 1800
-F 0 "U42" H 4500 1850 50  0000 C CNN
+F 0 "U40" H 4500 1850 50  0000 C CNN
 F 1 "74LS00" H 4500 1700 50  0000 C CNN
 F 2 "" H 4500 1800 50  0000 C CNN
 F 3 "" H 4500 1800 50  0000 C CNN
-	4    4500 1800
-	1    0    0    -1
-$EndComp
-$Comp
-L 74LS00 U45
-U 1 1 59303BAB
+	2    4500 1800
+	1    0    0    -1
+$EndComp
+$Comp
+L 74LS00 U40
+U 3 1 59303BAB
 P 5950 1800
-F 0 "U45" H 5950 1850 50  0000 C CNN
+F 0 "U40" H 5950 1850 50  0000 C CNN
 F 1 "74LS00" H 5950 1700 50  0000 C CNN
 F 2 "" H 5950 1800 50  0000 C CNN
 F 3 "" H 5950 1800 50  0000 C CNN
-	1    5950 1800
+	3    5950 1800
 	1    0    0    -1
 $EndComp
@@
 ~t5
 $Comp
-L SW_Push SW7
+L SW_Push SW5
 U 1 1 59305526
 P 1550 1250
-F 0 "SW7" H 1600 1350 50  0000 L CNN
+F 0 "SW5" H 1600 1350 50  0000 L CNN
 F 1 "SW_Push" H 1550 1190 50  0000 C CNN
 F 2 "" H 1550 1450 50  0000 C CNN
@@
 $EndComp
 $Comp
-L VCC #PWR067
+L VCC #PWR54
 U 1 1 5930559F
 P 1300 1050
-F 0 "#PWR067" H 1300 900 50  0001 C CNN
+F 0 "#PWR54" H 1300 900 50  0001 C CNN
 F 1 "VCC" H 1300 1200 50  0000 C CNN
 F 2 "" H 1300 1050 50  0000 C CNN
@@
 $EndComp
 $Comp
-L GND #PWR068
+L GND #PWR56
 U 1 1 5930575C
 P 1950 1650
-F 0 "#PWR068" H 1950 1400 50  0001 C CNN
+F 0 "#PWR56" H 1950 1400 50  0001 C CNN
 F 1 "GND" H 1950 1500 50  0000 C CNN
 F 2 "" H 1950 1650 50  0000 C CNN
@@
 ~RESET
 $Comp
-L R R29
+L R R23
 U 1 1 59305C2D
 P 1950 1450
-F 0 "R29" V 2030 1450 50  0000 C CNN
+F 0 "R23" V 2030 1450 50  0000 C CNN
 F 1 "1K" V 1950 1450 50  0000 C CNN
 F 2 "" V 1880 1450 50  0000 C CNN
@@
 Reset
 $Comp
-L VCC #PWR069
+L VCC #PWR63
 U 1 1 5ACBD5E7
 P 6300 5000
-F 0 "#PWR069" H 6300 4850 50  0001 C CNN
+F 0 "#PWR63" H 6300 4850 50  0001 C CNN
 F 1 "VCC" H 6300 5150 50  0000 C CNN
 F 2 "" H 6300 5000 50  0000 C CNN
@@
 	2700 5350 2700 5450
 $Comp
-L GND #PWR070
+L GND #PWR57
 U 1 1 5AD4813A
 P 2450 5100
-F 0 "#PWR070" H 2450 4850 50  0001 C CNN
+F 0 "#PWR57" H 2450 4850 50  0001 C CNN
 F 1 "GND" H 2450 4950 50  0000 C CNN
 F 2 "" H 2450 5100 50  0000 C CNN

Commit message: design as built
Parts:
- added RN?: R_Network08, Resistors_ThroughHole:Resistor_Array_SIP9, symbol R_Network08
- D1001: renamed from D36; footprint (none) -> LEDs:LED-5MM
- D1002: renamed from D37; footprint (none) -> LEDs:LED-5MM
- D1003: renamed from D38; footprint (none) -> LEDs:LED-5MM
- D1004: renamed from D39; footprint (none) -> LEDs:LED-5MM
- D1005: renamed from D40; footprint (none) -> LEDs:LED-5MM
- D1006: renamed from D41; footprint (none) -> LEDs:LED-5MM
- D1007: renamed from D42; footprint (none) -> LEDs:LED-5MM
- D1008: renamed from D43; footprint (none) -> LEDs:LED-5MM
- R1001: renamed from R23; footprint (none) -> Resistors_THT:Resistor_Horizontal_RM7mm
- SW1001: renamed from SW5; footprint (none) -> Buttons_Switches_THT:SW_PUSH_6mm_h9.5mm
- U1002: renamed from U33; footprint (none) -> Housings_DIP:DIP-14_W7.62mm_LongPads
- U1005: renamed from U40; footprint (none) -> Housings_DIP:DIP-14_W7.62mm_LongPads
- renumbered U37 to U1001, U38 to U1003, U39 to U1004, U41 to U1006
Connections:
- wire segments 109 -> 116
Other:
- moved on the sheet: D1001, D1002, D1003, D1004, D1005, D1006, D1007, D1008

Commit message: Update to current kicad version
Parts:
- removed D1001, D1002, D1003, D1004, D1005, D1006, D1007, D1008: LED, LEDs:LED-5MM, symbol LED
- removed R1001: 1K, Resistors_THT:Resistor_Horizontal_RM7mm, symbol R
- removed RN?: R_Network08, Resistors_ThroughHole:Resistor_Array_SIP9, symbol R_Network08
- removed SW1001: SW_Push, Buttons_Switches_THT:SW_PUSH_6mm_h9.5mm, symbol SW_Push
- removed U1001: 74LS161, Housings_DIP:DIP-16_W7.62mm_LongPads, symbol 74LS161
- removed U1002, U1005: 74LS00, Housings_DIP:DIP-14_W7.62mm_LongPads, symbol 74LS00
- removed U1003, U1006: 28C16, Housings_DIP:DIP-24_W15.24mm_LongPads, symbol 28C16
- removed U1004: 74LS138, Housings_DIP:DIP-16_W7.62mm_LongPads, symbol 74LS138
- added BAR7: HDSP-4830_2, Display:HDSP-4830, symbol LED:HDSP-4830_2
- added R18: 1K, symbol Device:R
- added RN9: 1K, Resistor_THT:R_Array_SIP9, symbol Device:R_Network08
- added SW7: Reset, symbol Switch:SW_Push
- added U32: 74LS00, symbol 74xx:74LS00
- added U33, U35: 28C16, symbol sap:28C16
- added U34: 74LS161, symbol 74xx:74LS161
- added U36: 74LS138, symbol 74xx:74LS138
Connections:
- wire segments 116 -> 97
Other:
- note removed: "Reset"
