File: kicad/control.sch (KiCad schematic (older format))
At the start: 16 parts, among them SW7 SW_Push, U24 74LS161, U25 28C16, U26 74LS138, U27 28C16, U42 74LS00, U45 74LS00

Commit message: Update to current kicad libraries
Parts:
- removed D59, D60, D61, D62, D63, D64, D65, D66: LED, symbol LED
- removed R29: 1K, symbol R
- removed SW7: SW_Push, symbol SW_Push
- removed U24: 74LS161, Housings_DIP:DIP-16_W7.62mm_LongPads, symbol 74LS161
- removed U25, U27: 28C16, Housings_DIP:DIP-24_W15.24mm_LongPads, symbol 28C16
- removed U26: 74LS138, Housings_DIP:DIP-16_W7.62mm_LongPads, symbol 74LS138
- removed U42, U45: 74LS00, symbol 74LS00
- added D30, D31, D32, D33, D34, D35, D36, D37: LED, symbol Device:LED
- added R12: 1K, symbol Device:R
- added SW5: Reset, symbol Switch:SW_Push
- added U37: 74LS00, symbol 74xx:74LS00
- added U38: 74LS161, symbol 74xx:74LS161
- added U39, U41: 28C16, symbol sap-be:28C16
- added U40: 74LS138, symbol 74xx:74LS138
Connections:
- wire segments 109 -> 124

Commit message: update bus names and improve sheet text
Parts:
- U48: renamed from U39; symbol sap-be:28C16 -> sap:28C16
- U50: renamed from U41; symbol sap-be:28C16 -> sap:28C16
- renumbered D30 to D46, D31 to D47, D32 to D48, D33 to D49, D34 to D50, D35 to D51, D36 to D52, D37 to D53, R12 to R14, SW5 to SW7, U37 to U46, U38 to U47, U40 to U49
Connections:
- net labels added: ir4, ir5, ir6, ir7, ir[0..7]
- net labels removed: i4, i5, i6, i7, i[0..7]
