File: kicad/instructionregister.sch (KiCad schematic (older format))
At the start: 11 parts, among them U15 74LS173, U16 74LS173, U17 74LS245

Commit message: bugfixed design
Parts:
- renumbered D22 to D44, D23 to D45, D24 to D46, D25 to D47, D26 to D48, D27 to D49, D28 to D50, D29 to D51, U15 to U42, U16 to U43, U17 to U44
Changed lines of the file:
@@
 LIBS:valves
 LIBS:switches
-LIBS:74xxx
-LIBS:28c16
 LIBS:sap-be-cache
-EELAYER 24 0
+EELAYER 25 0
 EELAYER END
 $Descr A4 11693 8268
@@
 $EndDescr
 $Comp
-L 74LS173 U15
+L 74LS173 U42
 U 1 1 5914399E
 P 4950 2400
-F 0 "U15" H 5050 2500 50  0000 C CNN
+F 0 "U42" H 5050 2500 50  0000 C CNN
 F 1 "74LS173" H 5050 2350 50  0000 C CNN
 F 2 "Housings_DIP:DIP-16_W7.62mm_LongPads" H 4950 2400 50  0001 C CNN
@@
 $EndComp
 $Comp
-L 74LS173 U16
+L 74LS173 U43
 U 1 1 5914399F
 P 4950 4400
-F 0 "U16" H 5050 4500 50  0000 C CNN
+F 0 "U43" H 5050 4500 50  0000 C CNN
 F 1 "74LS173" H 5050 4350 50  0000 C CNN
 F 2 "Housings_DIP:DIP-16_W7.62mm_LongPads" H 4950 4400 50  0001 C CNN
@@
 $EndComp
 $Comp
-L 74LS245 U17
+L 74LS245 U44
 U 1 1 590A460B
 P 7250 3350
-F 0 "U17" H 7350 3925 50  0000 L BNN
+F 0 "U44" H 7350 3925 50  0000 L BNN
 F 1 "74LS245" H 7300 2775 50  0000 L TNN
 F 2 "Housings_DIP:DIP-20_W7.62mm_LongPads" H 7250 3350 50  0001 C CNN
@@
 	3700 2050 3800 2150
 $Comp
-L VCC #PWR071
+L VCC #PWR70
 U 1 1 590A466E
 P 6450 3750
-F 0 "#PWR071" H 6450 3600 50  0001 C CNN
+F 0 "#PWR70" H 6450 3600 50  0001 C CNN
 F 1 "VCC" H 6450 3900 50  0000 C CNN
 F 2 "" H 6450 3750 50  0000 C CNN
@@
 ~LOAD
 $Comp
-L LED D22
+L LED D44
 U 1 1 590B2566
 P 6300 4900
-F 0 "D22" H 6300 5000 50  0000 C CNN
+F 0 "D44" H 6300 5000 50  0000 C CNN
 F 1 "LED" H 6300 4800 50  0000 C CNN
 F 2 "LEDs:LED-5MM" H 6300 4900 50  0001 C CNN
@@
 $EndComp
 $Comp
-L LED D23
+L LED D45
 U 1 1 591439A3
 P 6600 4900
-F 0 "D23" H 6600 5000 50  0000 C CNN
+F 0 "D45" H 6600 5000 50  0000 C CNN
 F 1 "LED" H 6600 4800 50  0000 C CNN
 F 2 "LEDs:LED-5MM" H 6600 4900 50  0001 C CNN
@@
 $EndComp
 $Comp
-L LED D24
+L LED D46
 U 1 1 591439A4
 P 6900 4900
-F 0 "D24" H 6900 5000 50  0000 C CNN
+F 0 "D46" H 6900 5000 50  0000 C CNN
 F 1 "LED" H 6900 4800 50  0000 C CNN
 F 2 "LEDs:LED-5MM" H 6900 4900 50  0001 C CNN
@@
 $EndComp
 $Comp
-L LED D25
+L LED D47
 U 1 1 590B27C9
 P 7200 4900
-F 0 "D25" H 7200 5000 50  0000 C CNN
+F 0 "D47" H 7200 5000 50  0000 C CNN
 F 1 "LED" H 7200 4800 50  0000 C CNN
 F 2 "LEDs:LED-5MM" H 7200 4900 50  0001 C CNN
@@
 $EndComp
 $Comp
-L LED D26
+L LED D48
 U 1 1 590B28D2
 P 7500 4900
-F 0 "D26" H 7500 5000 50  0000 C CNN
+F 0 "D48" H 7500 5000 50  0000 C CNN
 F 1 "LED" H 7500 4800 50  0000 C CNN
 F 2 "LEDs:LED-5MM" H 7500 4900 50  0001 C CNN
@@
 $EndComp
 $Comp
-L LED D27
+L LED D49
 U 1 1 590B2981
 P 7800 4900
-F 0 "D27" H 7800 5000 50  0000 C CNN
+F 0 "D49" H 7800 5000 50  0000 C CNN
 F 1 "LED" H 7800 4800 50  0000 C CNN
 F 2 "LEDs:LED-5MM" H 7800 4900 50  0001 C CNN
@@
 $EndComp
 $Comp
-L LED D28
+L LED D50
 U 1 1 590B29B6
 P 8100 4900
-F 0 "D28" H 8100 5000 50  0000 C CNN
+F 0 "D50" H 8100 5000 50  0000 C CNN
 F 1 "LED" H 8100 4800 50  0000 C CNN
 F 2 "LEDs:LED-5MM" H 8100 4900 50  0001 C CNN
@@
 $EndComp
 $Comp
-L LED D29
+L LED D51
 U 1 1 590B29E1
 P 8400 4900
-F 0 "D29" H 8400 5000 50  0000 C CNN
+F 0 "D51" H 8400 5000 50  0000 C CNN
 F 1 "LED" H 8400 4800 50  0000 C CNN
 F 2 "LEDs:LED-5MM" H 8400 4900 50  0001 C CNN
@@
 ~LOAD
 $Comp
-L GND #PWR072
+L GND #PWR71
 U 1 1 590D3ED6
 P 8650 5250
-F 0 "#PWR072" H 8650 5000 50  0001 C CNN
+F 0 "#PWR71" H 8650 5000 50  0001 C CNN
 F 1 "GND" H 8650 5100 50  0000 C CNN
 F 2 "" H 8650 5250 50  0000 C CNN
@@
 r[0..7]
 $Comp
-L GND #PWR073
+L GND #PWR69
 U 1 1 59133E3E
 P 6250 3550
-F 0 "#PWR073" H 6250 3300 50  0001 C CNN
+F 0 "#PWR69" H 6250 3300 50  0001 C CNN
 F 1 "GND" H 6250 3400 50  0000 C CNN
 F 2 "" H 6250 3550 50  0000 C CNN

Commit message: design as built
Parts:
- renumbered D44 to D701, D45 to D702, D46 to D703, D47 to D704, D48 to D705, D49 to D706, D50 to D707, D51 to D708, U42 to U701, U43 to U702, U44 to U703
Connections:
- wire segments 74 -> 73
Changed lines of the file:
@@
 LIBS:valves
 LIBS:switches
+LIBS:74xxx
+LIBS:28c16
+LIBS:ne556
 LIBS:sap-be-cache
 EELAYER 25 0
@@
 $Descr A4 11693 8268
 encoding utf-8
-Sheet 10 12
+Sheet 7 12
 Title "Simple As Possible computer by Ben Eater"
-Date "2017-05-10"
-Rev "1"
+Date "2018-06-03"
+Rev "2"
 Comp "Schematic released as CC BY-SA"
 Comment1 "Schematic capture by Vincent Sanders"
@@
 $EndDescr
 $Comp
-L 74LS173 U42
+L 74LS173 U701
 U 1 1 5914399E
 P 4950 2400
-F 0 "U42" H 5050 2500 50  0000 C CNN
+F 0 "U701" H 5050 2500 50  0000 C CNN
 F 1 "74LS173" H 5050 2350 50  0000 C CNN
 F 2 "Housings_DIP:DIP-16_W7.62mm_LongPads" H 4950 2400 50  0001 C CNN
@@
 $EndComp
 $Comp
-L 74LS173 U43
+L 74LS173 U702
 U 1 1 5914399F
 P 4950 4400
-F 0 "U43" H 5050 4500 50  0000 C CNN
+F 0 "U702" H 5050 4500 50  0000 C CNN
 F 1 "74LS173" H 5050 4350 50  0000 C CNN
 F 2 "Housings_DIP:DIP-16_W7.62mm_LongPads" H 4950 4400 50  0001 C CNN
@@
 $EndComp
 $Comp
-L 74LS245 U44
+L 74LS245 U703
 U 1 1 590A460B
 P 7250 3350
-F 0 "U44" H 7350 3925 50  0000 L BNN
+F 0 "U703" H 7350 3925 50  0000 L BNN
 F 1 "74LS245" H 7300 2775 50  0000 L TNN
 F 2 "Housings_DIP:DIP-20_W7.62mm_LongPads" H 7250 3350 50  0001 C CNN
@@
 	6000 2150 6100 2250
 Text Label 6550 2850 0    60   ~ 0
+r7
+Text Label 6550 2950 0    60   ~ 0
+r6
+Text Label 6550 3050 0    60   ~ 0
+r5
+Text Label 6550 3150 0    60   ~ 0
+r4
+Text Label 6550 3250 0    60   ~ 0
+r3
+Text Label 6550 3350 0    60   ~ 0
+r2
+Text Label 6550 3450 0    60   ~ 0
+r1
+Text Label 6550 3550 0    60   ~ 0
 r0
-Text Label 6550 2950 0    60   ~ 0
-r1
-Text Label 6550 3050 0    60   ~ 0
-r2
-Text Label 6550 3150 0    60   ~ 0
-r3
-Text Label 6550 3250 0    60   ~ 0
-r4
-Text Label 6550 3350 0    60   ~ 0
-r5
-Text Label 6550 3450 0    60   ~ 0
-r6
-Text Label 6550 3550 0    60   ~ 0
-r7
 Entry Wire Line
 	6100 2750 6200 2850
@@
 	3700 2050 3800 2150
 $Comp
-L VCC #PWR70
+L VCC #PWR036
 U 1 1 590A466E
 P 6450 3750
-F 0 "#PWR70" H 6450 3600 50  0001 C CNN
+F 0 "#PWR036" H 6450 3600 50  0001 C CNN
 F 1 "VCC" H 6450 3900 50  0000 C CNN
 F 2 "" H 6450 3750 50  0000 C CNN
@@
 ~LOAD
 $Comp
-L LED D44
+L LED D701
 U 1 1 590B2566
 P 6300 4900
-F 0 "D44" H 6300 5000 50  0000 C CNN
+F 0 "D701" H 6300 5000 50  0000 C CNN
 F 1 "LED" H 6300 4800 50  0000 C CNN
 F 2 "LEDs:LED-5MM" H 6300 4900 50  0001 C CNN
@@
 $EndComp
 $Comp
-L LED D45
+L LED D702
 U 1 1 591439A3
 P 6600 4900
-F 0 "D45" H 6600 5000 50  0000 C CNN
+F 0 "D702" H 6600 5000 50  0000 C CNN
 F 1 "LED" H 6600 4800 50  0000 C CNN
 F 2 "LEDs:LED-5MM" H 6600 4900 50  0001 C CNN
@@
 $EndComp
 $Comp
-L LED D46
+L LED D703
 U 1 1 591439A4
 P 6900 4900
-F 0 "D46" H 6900 5000 50  0000 C CNN
+F 0 "D703" H 6900 5000 50  0000 C CNN
 F 1 "LED" H 6900 4800 50  0000 C CNN
 F 2 "LEDs:LED-5MM" H 6900 4900 50  0001 C CNN
@@
 $EndComp
 $Comp
-L LED D47
+L LED D704
 U 1 1 590B27C9
 P 7200 4900
-F 0 "D47" H 7200 5000 50  0000 C CNN
+F 0 "D704" H 7200 5000 50  0000 C CNN
 F 1 "LED" H 7200 4800 50  0000 C CNN
 F 2 "LEDs:LED-5MM" H 7200 4900 50  0001 C CNN
@@
 $EndComp
 $Comp
-L LED D48
+L LED D705
 U 1 1 590B28D2
 P 7500 4900
-F 0 "D48" H 7500 5000 50  0000 C CNN
+F 0 "D705" H 7500 5000 50  0000 C CNN
 F 1 "LED" H 7500 4800 50  0000 C CNN
 F 2 "LEDs:LED-5MM" H 7500 4900 50  0001 C CNN
@@
 $EndComp
 $Comp
-L LED D49
+L LED D706
 U 1 1 590B2981
 P 7800 4900
-F 0 "D49" H 7800 5000 50  0000 C CNN
+F 0 "D706" H 7800 5000 50  0000 C CNN
 F 1 "LED" H 7800 4800 50  0000 C CNN
 F 2 "LEDs:LED-5MM" H 7800 4900 50  0001 C CNN
@@
 $EndComp
 $Comp
-L LED D50
+L LED D707
 U 1 1 590B29B6
 P 8100 4900
-F 0 "D50" H 8100 5000 50  0000 C CNN
+F 0 "D707" H 8100 5000 50  0000 C CNN
 F 1 "LED" H 8100 4800 50  0000 C CNN
 F 2 "LEDs:LED-5MM" H 8100 4900 50  0001 C CNN
@@
 $EndComp
 $Comp
-L LED D51
+L LED D708
 U 1 1 590B29E1
 P 8400 4900
-F 0 "D51" H 8400 5000 50  0000 C CNN
+F 0 "D708" H 8400 5000 50  0000 C CNN
 F 1 "LED" H 8400 4800 50  0000 C CNN
 F 2 "LEDs:LED-5MM" H 8400 4900 50  0001 C CNN
@@
 ~LOAD
 $Comp
-L GND #PWR71
+L GND #PWR037
 U 1 1 590D3ED6
 P 8650 5250
-F 0 "#PWR71" H 8650 5000 50  0001 C CNN
+F 0 "#PWR037" H 8650 5000 50  0001 C CNN
 F 1 "GND" H 8650 5100 50  0000 C CNN
 F 2 "" H 8650 5250 50  0000 C CNN
@@
 w[0..7]
 Text Label 8150 2850 0    60   ~ 0
+w7
+Text Label 8150 2950 0    60   ~ 0
+w6
+Text Label 8150 3050 0    60   ~ 0
+w5
+Text Label 8150 3150 0    60   ~ 0
+w4
+Text Label 8150 3250 0    60   ~ 0
+w3
+Text Label 8150 3350 0    60   ~ 0
+w2
+Text Label 8150 3450 0    60   ~ 0
+w1
+Text Label 8150 3550 0    60   ~ 0
 w0
-Text Label 8150 2950 0    60   ~ 0
-w1
-Text Label 8150 3050 0    60   ~ 0
-w2
-Text Label 8150 3150 0    60   ~ 0
-w3
-Text Label 8150 3250 0    60   ~ 0
-w4
-Text Label 8150 3350 0    60   ~ 0
-w5
-Text Label 8150 3450 0    60   ~ 0
-w6
-Text Label 8150 3550 0    60   ~ 0
-w7
 Text Label 4100 1850 0    60   ~ 0
 w0
@@
 Text HLabel 6650 5600 2    60   Output ~ 0
 r[0..7]
-$Comp
-L GND #PWR69
-U 1 1 59133E3E
-P 6250 3550
-F 0 "#PWR69" H 6250 3300 50  0001 C CNN
-F 1 "GND" H 6250 3400 50  0000 C CNN
-F 2 "" H 6250 3550 50  0000 C CNN
-F 3 "" H 6250 3550 50  0000 C CNN
-	1    6250 3550
-	1    0    0    -1
-$EndComp
-Wire Wire Line
-	6250 3250 6250 3550
-Connection ~ 6250 3450
-Connection ~ 6250 3350
-Wire Wire Line
-	6550 3250 6250 3250
-Wire Wire Line
-	6550 3350 6250 3350
-Wire Wire Line
-	6550 3450 6250 3450
-Wire Wire Line
-	6250 3550 6550 3550
+Wire Wire Line
+	6200 3250 6550 3250
+Wire Wire Line
+	6200 3350 6550 3350
+Wire Wire Line
+	6200 3450 6550 3450
+Wire Wire Line
+	6200 3550 6550 3550
 Text HLabel 2750 2350 0    60   Input ~ 0
 RESET
+Entry Wire Line
+	6100 3150 6200 3250
+Entry Wire Line
+	6100 3250 6200 3350
+Entry Wire Line
+	6100 3350 6200 3450
+Entry Wire Line
+	6100 3450 6200 3550
 $EndSCHEMATC

Commit message: Update to current kicad version
Parts:
- removed D701, D702, D703, D704, D705, D706, D707, D708: LED, LEDs:LED-5MM, symbol LED
- removed U701, U702: 74LS173, Housings_DIP:DIP-16_W7.62mm_LongPads, symbol 74LS173
- removed U703: 74LS245, Housings_DIP:DIP-20_W7.62mm_LongPads, symbol 74LS245
- added BAR5: HDSP-4830_2, Display:HDSP-4830, symbol LED:HDSP-4830_2
- added RN7: 1K, Resistor_THT:R_Array_SIP9, symbol Device:R_Network08
- added U23: 74LS245, symbol 74xx:74LS245
- added U24, U25: 74LS173, symbol 74xx:74LS173
Connections:
- net labels added: ir0, ir1, ir2, ir3, ir4, ir5, ir6, ir7, ir[0..7]
- net labels removed: r0, r1, r2, r3, r4, r5, r6, r7, r[0..7], ~RENABLE
- wire segments 73 -> 68
- no-connect marks 0 -> 4
