File: kicad/memory.sch (KiCad schematic (older format))
At the start: 33 parts, among them SW3 SW_DIP_x08, SW5 SW_DIP_x04, U32 74LS04, U35 74LS173, U36 74LS157, U37 74LS157, U38 74LS189, U39 74LS189, U40 74LS157, U41 74LS04, U42 74LS00, U43 74LS245, U44 74LS157

Commit message: bugfixed design
Parts:
- removed C8: 0.1u, Capacitors_THT:C_Disc_D6_P5, symbol C
- removed D45, D46, D47, D48, D50: LED, LEDs:LED-5MM, symbol LED
- removed R26, R27: 220, Resistors_THT:Resistor_Horizontal_RM7mm, symbol R
- removed R28: 1K, Resistors_THT:Resistor_Horizontal_RM7mm, symbol R
- removed SW-PGM1: SW_SPDT, Buttons_Switches_THT:SW_Micro_SPST, symbol SW_SPDT
- removed SW-WR1: SW_Push, Buttons_Switches_THT:SW_PUSH_6mm_h9.5mm, symbol SW_Push
- removed SW3: SW_DIP_x08, Buttons_Switches_THT:SW_DIP_x8_Slide, symbol SW_DIP_x08
- removed SW5: SW_DIP_x04, Buttons_Switches_THT:SW_DIP_x4_Slide, symbol SW_DIP_x04
- removed U32: 74LS04, Housings_DIP:DIP-14_W7.62mm_LongPads, symbol 74LS04
- removed U38, U39: 74LS189, Housings_DIP:DIP-16_W7.62mm_LongPads, symbol 74LS189
- removed U40: 74LS157, Housings_DIP:DIP-16_W7.62mm_LongPads, symbol 74LS157
- removed unit 1 of U41
- removed unit 5 of U41
- removed unit 2 of U41
- removed unit 3 of U41
- removed U42: 74LS00, Housings_DIP:DIP-14_W7.62mm_LongPads, symbol 74LS00
- removed U43: 74LS245, Housings_DIP:DIP-20_W7.62mm_LongPads, symbol 74LS245
- added C10: 0.1u, Capacitors_THT:C_Disc_D6_P5, symbol C
- added D84, D85, D87, D96, D97: LED, LEDs:LED-5MM, symbol LED
- added R43: 1K, Resistors_THT:Resistor_Horizontal_RM7mm, symbol R
- added R44, R45: 220, Resistors_THT:Resistor_Horizontal_RM7mm, symbol R
- added R46: 4k7, Resistors_THT:Resistor_Horizontal_RM7mm, symbol R
- added SW-PGM3: SW_SPDT, Buttons_Switches_THT:SW_Micro_SPST, symbol SW_SPDT
- added SW-WR3: SW_Push, Buttons_Switches_THT:SW_PUSH_6mm_h9.5mm, symbol SW_Push
- added SW8: SW_DIP_x04, Buttons_Switches_THT:SW_DIP_x4_Slide, symbol SW_DIP_x04
- added SW9: SW_DIP_x08, Buttons_Switches_THT:SW_DIP_x8_Slide, symbol SW_DIP_x08
- added U54, U65: 74LS04, Housings_DIP:DIP-14_W7.62mm_LongPads, symbol 74LS04
- added U60, U61: 74LS189, Housings_DIP:DIP-16_W7.62mm_LongPads, symbol 74LS189
- added U62: 74LS00, symbol 74LS00
- added U63: 74LS157, Housings_DIP:DIP-16_W7.62mm_LongPads, symbol 74LS157
- added unit 1 of U64
- added unit 5 of U64
- added unit 2 of U64
- added unit 6 of U64
- added unit 3 of U64
- added U66: 74LS245, Housings_DIP:DIP-20_W7.62mm_LongPads, symbol 74LS245
- renumbered D49 to D86, D51 to D88, D52 to D89, D53 to D90, D54 to D91, D55 to D92, D56 to D93, D57 to D94, D58 to D95, U35 to U57, U36 to U58, U37 to U59, U41 to U64, U44 to U67
Connections:
- wire segments 242 -> 246
Other:
- moved on the sheet: D86, D88, D89, D90, D91, D92, D93, D94, D95

Commit message: design as built
Parts:
- removed C10: 0.1u, Capacitors_THT:C_Disc_D6_P5, symbol C
- removed D84, D85, D86, D87, D88, D89, D90, D91, D92, D93, D94, D95, D96, D97: LED, LEDs:LED-5MM, symbol LED
- removed R43: 1K, Resistors_THT:Resistor_Horizontal_RM7mm, symbol R
- removed R44, R45: 220, Resistors_THT:Resistor_Horizontal_RM7mm, symbol R
- removed R46: 4k7, Resistors_THT:Resistor_Horizontal_RM7mm, symbol R
- removed SW-PGM3: SW_SPDT, Buttons_Switches_THT:SW_Micro_SPST, symbol SW_SPDT
- removed SW-WR3: SW_Push, Buttons_Switches_THT:SW_PUSH_6mm_h9.5mm, symbol SW_Push
- removed SW8: SW_DIP_x04, Buttons_Switches_THT:SW_DIP_x4_Slide, symbol SW_DIP_x04
- removed SW9: SW_DIP_x08, Buttons_Switches_THT:SW_DIP_x8_Slide, symbol SW_DIP_x08
- removed U54, U64, U65: 74LS04, Housings_DIP:DIP-14_W7.62mm_LongPads, symbol 74LS04
- removed U57: 74LS173, Housings_DIP:DIP-16_W7.62mm_LongPads, symbol 74LS173
- removed U58, U59, U63, U67: 74LS157, Housings_DIP:DIP-16_W7.62mm_LongPads, symbol 74LS157
- removed U60, U61: 74LS189, Housings_DIP:DIP-16_W7.62mm_LongPads, symbol 74LS189
- removed U62: 74LS00, symbol 74LS00
- removed U66: 74LS245, Housings_DIP:DIP-20_W7.62mm_LongPads, symbol 74LS245
- added C201: 100n, Capacitors_THT:C_Disc_D6_P5, symbol C
- added D201, D202, D203, D204, D205, D206, D207, D208, D209, D210, D211, D212: LED, LEDs:LED-5MM, symbol LED
- added D213: PGM LED, LEDs:LED-5MM, symbol LED
- added D214: RUN LED, LEDs:LED-5MM, symbol LED
- added R201, R203, R204: 1K, Resistors_THT:Resistor_Horizontal_RM7mm, symbol R
- added R202: 1k, Resistors_THT:Resistor_Horizontal_RM7mm, symbol R
- added RN201, RN202, RN203: 1K, Resistors_ThroughHole:Resistor_Array_SIP9, symbol R_Network08
- added SW-PGM201: SW_Mode, Buttons_Switches_THT:SW_Micro_SPST, symbol SW_SPDT
- added SW-WR201: SW_Write, Buttons_Switches_THT:SW_PUSH_6mm_h9.5mm, symbol SW_Push
- added SW201: SW_DIP_x08, Buttons_Switches_THT:SW_DIP_x8_Slide, symbol SW_DIP_x08
- added SW202: SW_DIP_x04, Buttons_Switches_THT:SW_DIP_x4_Slide, symbol SW_DIP_x04
- added U201, U208: 74LS245, symbol 74LS245
- added U202: 74LS173, Housings_DIP:DIP-16_W7.62mm_LongPads, symbol 74LS173
- added U203, U204, U209: 74LS157, Housings_DIP:DIP-16_W7.62mm_LongPads, symbol 74LS157
- added U205, U206: 74F219, symbol 74F219
- added U207: 74LS00, symbol 74LS00
Connections:
- net labels added: ~CLK, ~PGM
- wire segments 246 -> 245
- no-connect marks 9 -> 17

Commit message: Update to current kicad version
Parts:
- removed C201: 100n, Capacitors_THT:C_Disc_D6_P5, symbol C
- removed D201, D202, D203, D204, D205, D206, D207, D208, D209, D210, D211, D212: LED, LEDs:LED-5MM, symbol LED
- removed D213: PGM LED, LEDs:LED-5MM, symbol LED
- removed D214: RUN LED, LEDs:LED-5MM, symbol LED
- removed R201, R203, R204: 1K, Resistors_THT:Resistor_Horizontal_RM7mm, symbol R
- removed R202: 1k, Resistors_THT:Resistor_Horizontal_RM7mm, symbol R
- removed RN201, RN202, RN203: 1K, Resistors_ThroughHole:Resistor_Array_SIP9, symbol R_Network08
- removed SW-PGM201: SW_Mode, Buttons_Switches_THT:SW_Micro_SPST, symbol SW_SPDT
- removed SW-WR201: SW_Write, Buttons_Switches_THT:SW_PUSH_6mm_h9.5mm, symbol SW_Push
- removed SW201: SW_DIP_x08, Buttons_Switches_THT:SW_DIP_x8_Slide, symbol SW_DIP_x08
- removed SW202: SW_DIP_x04, Buttons_Switches_THT:SW_DIP_x4_Slide, symbol SW_DIP_x04
- removed U201, U208: 74LS245, symbol 74LS245
- removed U202: 74LS173, Housings_DIP:DIP-16_W7.62mm_LongPads, symbol 74LS173
- removed U203, U204, U209: 74LS157, Housings_DIP:DIP-16_W7.62mm_LongPads, symbol 74LS157
- removed U205, U206: 74F219, symbol 74F219
- removed U207: 74LS00, symbol 74LS00
- added BAR4: HDSP-4830_2, Display:HDSP-4830, symbol LED:HDSP-4830_2
- added C1, C3: 100nF, symbol Device:C
- added C2: 10nF, symbol Device:C
- added C4: 330nF, symbol Device:C
- added R3: 10K, symbol Device:R
- added R4: 1M, symbol Device:R
- added R5, R6: 1K, symbol Device:R
- added RN5: 1k, Resistor_THT:R_Array_SIP9, symbol Device:R_Network08
- added RN6: 1K, Resistor_THT:R_Array_SIP9, symbol Device:R_Network08
- added SW3: Data, symbol Switch:SW_DIP_x08
- added SW4: Write, symbol Switch:SW_Push
- added U10: CY7C199, symbol Memory_RAM:CY7C199
- added U11, U9: 74LS245, symbol 74xx:74LS245
- added U12, U13: 74LS00, symbol 74xx:74LS00
- added U14: LM555, symbol Timer:LM555
- added U15: 74LS157, symbol 74xx:74LS157
Connections:
- net labels added: PGMWRITE, mb0, mb1, mb2, mb3, mb4, mb5, mb6, mb7, mb[0..7], ~BEN, ~OE, ~PGMWRITE, ~READ, ~RUNBEN, ~RUNWE, ~SE
- net labels removed: CLR, RESET, d0, d1, d2, d3, d4, d5, d6, d7, m0, m1, m2, m3, m4, m5, m6, m7, ~ALOAD, ~CLK, ~PGM, ~WENABLE
- wire segments 245 -> 176
- no-connect marks 17 -> 7
