File: kicad/memory.sch (KiCad schematic (older format))
At the start: 35 parts, among them SW8 SW_DIP_x04, SW9 SW_DIP_x08, U54 74LS04, U57 74LS173, U58 74LS157, U59 74LS157, U60 74LS189, U61 74LS189, U62 74LS00, U63 74LS157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

Commit message: Update bugfix version to use updated kicad libraries
Parts:
- removed C10: 0.1u, Capacitors_THT:C_Disc_D6_P5, symbol C
- removed D84, D85, D86, D87, D88, D89, D90, D91, D92, D93, D94, D95, D96, D97: LED, LEDs:LED-5MM, symbol LED
- removed R43: 1K, Resistors_THT:Resistor_Horizontal_RM7mm, symbol R
- removed R44, R45: 220, Resistors_THT:Resistor_Horizontal_RM7mm, symbol R
- removed R46: 4k7, Resistors_THT:Resistor_Horizontal_RM7mm, symbol R
- removed SW-PGM3: SW_SPDT, Buttons_Switches_THT:SW_Micro_SPST, symbol SW_SPDT
- removed SW-WR3: SW_Push, Buttons_Switches_THT:SW_PUSH_6mm_h9.5mm, symbol SW_Push
- removed SW8: SW_DIP_x04, Buttons_Switches_THT:SW_DIP_x4_Slide, symbol SW_DIP_x04
- removed SW9: SW_DIP_x08, Buttons_Switches_THT:SW_DIP_x8_Slide, symbol SW_DIP_x08
- removed U54, U64, U65: 74LS04, Housings_DIP:DIP-14_W7.62mm_LongPads, symbol 74LS04
- removed U57: 74LS173, Housings_DIP:DIP-16_W7.62mm_LongPads, symbol 74LS173
- removed U58, U59, U63, U67: 74LS157, Housings_DIP:DIP-16_W7.62mm_LongPads, symbol 74LS157
- removed U60, U61: 74LS189, Housings_DIP:DIP-16_W7.62mm_LongPads, symbol 74LS189
- removed U62: 74LS00, symbol 74LS00
- removed U66: 74LS245, Housings_DIP:DIP-20_W7.62mm_LongPads, symbol 74LS245
- added C8: 100nF, symbol Device:C
- added D22, D23, D24, D25, D26, D27, D28, D29: LED, symbol Device:LED
- added R11: 1K, symbol Device:R
- added R?: 4K7, symbol Device:R
- added SW3: Data, symbol Switch:SW_DIP_x08
- added SW4: Write, symbol Switch:SW_Push
- added U28, U29, U36: 74LS157, symbol 74xx:74LS157
- added U31, U32: 74LS189, symbol sap-be:74LS189
- added U33, U34: 74LS04, symbol 74xx:74LS04
- added U35, U? (x2): 74LS00, symbol 74xx:74LS00
- added U?: 74LS240, symbol 74xx:74LS240
Connections:
- net labels removed: CLR, RESET, ~ALOAD
- wire segments 246 -> 165

Commit message: update kicad project name
Parts:
- U31, U32: symbol sap-be:74LS189 -> sap:74LS189
Changed lines of the file:
@@
 	1800 2900 1800 3950
 $Comp
-L sap-be:74LS189 U32
+L sap:74LS189 U32
 U 1 1 611DA12F
 P 4800 4750
@@
 $EndComp
 $Comp
-L sap-be:74LS189 U31
+L sap:74LS189 U31
 U 1 1 611D9751
 P 4800 2450
