File: kicad/output.sch (KiCad schematic (older format))
At the start: 14 parts, among them U18 74LS08, U19 NE555, U20 74LS273, U21 74LS76, U22 28C16, U23 74LS139

Commit message: bugfixed design
Parts:
- removed U18: 74LS08, Housings_DIP:DIP-14_W7.62mm_LongPads, symbol 74LS08
- added U22: 74HC74, symbol 74HC74
- renumbered C3 to C6, C4 to C7, R6 to R10, R5 to R9, U20 to U23, U22 to U24, U21 to U25, U23 to U26, U19 to U27
Connections:
- net labels added: OCLK
- wire segments 116 -> 120
- no-connect marks 2 -> 3
Other:
- moved on the sheet: AFF1, AFF2, AFF3, AFF4, C6, C7, R10, R9, U23, U24, U25A, U25B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

Commit message: design as built
Parts:
- removed AFF1, AFF2, AFF3, AFF4: LTS-6980HR, Displays_7-Segment:7SegmentLED_LTS6760_LTS6780, symbol LTS-6980HR
- removed C6, C7: 10n, Capacitors_THT:C_Disc_D6_P5, symbol C
- removed R10: 100K, Resistors_THT:Resistor_Horizontal_RM7mm, symbol R
- removed R9: 1K, Resistors_THT:Resistor_Horizontal_RM7mm, symbol R
- removed U22: 74HC74, symbol 74HC74
- removed U23: 74LS273, Housings_DIP:DIP-20_W7.62mm_LongPads, symbol 74LS273
- removed U27: NE555, Housings_DIP:DIP-8_W7.62mm_LongPads, symbol NE555
- added AFF1201: CC56-12, Displays_7-Segment:Cx56-12, symbol CC56-12
- added R1201, R1202, R1203, R1204, R1205, R1206, R1207, R1208: R, Resistors_THT:Resistor_Horizontal_RM7mm, symbol R
- added U1201: 74LS377, Housings_DIP:DIP-20_W7.62mm_LongPads, symbol 74LS377
- renumbered U25 to U1202, U24 to U1203, U26 to U1204
Connections:
- net labels removed: OCLK
- wire segments 120 -> 74
- no-connect marks 3 -> 2
Other:
- moved on the sheet: U1202A, U1202B, U1203, U1204A

Commit message: Update to current kicad version
Parts:
- removed AFF1201: CC56-12, Displays_7-Segment:Cx56-12, symbol CC56-12
- removed R1201, R1202, R1203, R1204, R1205, R1206, R1207, R1208: R, Resistors_THT:Resistor_Horizontal_RM7mm, symbol R
- removed U1201: 74LS377, Housings_DIP:DIP-20_W7.62mm_LongPads, symbol 74LS377
- removed U1202: 74LS76, Housings_DIP:DIP-16_W7.62mm_LongPads, symbol 74LS76
- removed U1203: 28C16, Housings_DIP:DIP-24_W15.24mm_LongPads, symbol 28C16
- removed U1204: 74LS139, Housings_DIP:DIP-16_W7.62mm_LongPads, symbol 74LS139
- added R35, R36, R37, R38, R39, R40, R41, R42: 680R, symbol Device:R
- added U39: 74LS139, symbol 74xx:74LS139
- added U40: 74LS112, symbol 74xx:74LS112
- added U41: 74LS377, symbol 74xx:74LS377
- added U42: 28C16, symbol sap:28C16
- added U43: CC56-12EWA, Display_7Segment:CA56-12EWA, symbol Display_Character:CC56-12EWA
Connections:
- net labels added: ~LOAD
- net labels removed: LOAD, s0, s1, s2, s3, s4, s5, s6, s7, ~CLR
- wire segments 74 -> 81
