File: kicad/output.sch (KiCad schematic (older format))
At the start: 14 parts, among them U18 74LS08, U19 NE555, U20 74LS273, U21 74LS76, U22 28C16, U23 74LS139

Commit message: Update to current kicad libraries
Parts:
- removed AFF1, AFF2, AFF3, AFF4: LTS-6980HR, Displays_7-Segment:7SegmentLED_LTS6760_LTS6780, symbol LTS-6980HR
- removed C3, C4: 10n, Capacitors_THT:C_Disc_D6_P5, symbol C
- removed R5: 1K, Resistors_THT:Resistor_Horizontal_RM7mm, symbol R
- removed R6: 100K, Resistors_THT:Resistor_Horizontal_RM7mm, symbol R
- removed U18: 74LS08, Housings_DIP:DIP-14_W7.62mm_LongPads, symbol 74LS08
- removed U19: NE555, Housings_DIP:DIP-8_W7.62mm_LongPads, symbol NE555
- removed U20: 74LS273, Housings_DIP:DIP-20_W7.62mm_LongPads, symbol 74LS273
- removed U21: 74LS76, Housings_DIP:DIP-16_W7.62mm_LongPads, symbol 74LS76
- removed U22: 28C16, Housings_DIP:DIP-24_W15.24mm_LongPads, symbol 28C16
- removed U23: 74LS139, Housings_DIP:DIP-16_W7.62mm_LongPads, symbol 74LS139
- added AFF1, AFF2, AFF3, AFF4: LTS-6980HR, Display_7Segment:7SegmentLED_LTS6760_LTS6780, symbol Display_Character:LTS-6980HR
- added C6, C7: 10n, symbol Device:C
- added R10: 1K, symbol Device:R
- added R9: 100K, symbol Device:R
- added U22: 74LS08, symbol 74xx:74LS08
- added U23: 74LS139, symbol 74xx:74LS139
- added U24: 74LS76, symbol 74xx:74LS76
- added U25: 74LS273, symbol 74xx:74LS273
- added U26: 28C16, symbol sap-be:28C16
- added U27: LM555, symbol Timer:LM555
Connections:
- wire segments 116 -> 143

Commit message: update bus names and improve sheet text
Parts:
- U44: renamed from U26; symbol sap-be:28C16 -> sap:28C16
- renumbered C6 to C7, C7 to C8, R9 to R12, R10 to R13, U22 to U33, U23 to U41, U24 to U42, U25 to U43, U27 to U45
Changed lines of the file:
@@
 encoding utf-8
 Sheet 7 13
-Title "Simple As Possible computer by Ben Eater"
+Title "Simple As Possible computer"
 Date "2017-05-10"
 Rev "1"
 Comp "Schematic released as CC BY-SA"
-Comment1 "Schematic capture by Vincent Sanders"
+Comment1 "Schematic capture by Vincent Sanders of a design by Ben Eater"
 Comment2 "7 segment output register"
 Comment3 ""
@@
 	9450 4300 9600 4300
 $Comp
-L 74xx:74LS139 U23
+L 74xx:74LS139 U41
 U 1 1 5F80E208
 P 9900 2550
-F 0 "U23" H 9900 2800 50  0000 C CNN
+F 0 "U41" H 9900 2800 50  0000 C CNN
 F 1 "74LS139" H 9900 2200 50  0000 C CNN
 F 2 "" H 9900 2550 50  0001 C CNN
@@
 $EndComp
 $Comp
-L 74xx:74LS139 U23
+L 74xx:74LS139 U41
 U 3 1 5F80F43A
 P 1400 6950
-F 0 "U23" V 1250 6850 50  0000 L CNN
+F 0 "U41" V 1250 6850 50  0000 L CNN
 F 1 "74LS139" V 1550 6800 50  0000 L CNN
 F 2 "" H 1400 6950 50  0001 C CNN
@@
 $EndComp
 $Comp
-L Timer:LM555 U27
+L Timer:LM555 U45
 U 1 1 5F8147A8
 P 6800 1350
-F 0 "U27" H 6550 1700 50  0000 C CNN
+F 0 "U45" H 6550 1700 50  0000 C CNN
 F 1 "LM555" H 7050 1000 50  0000 C CNN
 F 2 "" H 6800 1350 50  0001 C CNN
@@
 	9200 2750 9400 2750
 $Comp
-L 74xx:74LS76 U24
+L 74xx:74LS76 U42
 U 1 1 5F862F3C
 P 9450 1400
-F 0 "U24" H 9300 1650 50  0000 C CNN
+F 0 "U42" H 9300 1650 50  0000 C CNN
 F 1 "74LS76" H 9650 1150 50  0000 C CNN
 F 2 "" H 9450 1400 50  0001 C CNN
@@
 $EndComp
 $Comp
-L 74xx:74LS76 U24
+L 74xx:74LS76 U42
 U 2 1 5F864DF2
 P 10550 1400
-F 0 "U24" H 10400 1650 50  0000 C CNN
+F 0 "U42" H 10400 1650 50  0000 C CNN
 F 1 "74LS76" H 10700 1150 50  0000 C CNN
 F 2 "" H 10550 1400 50  0001 C CNN
@@
 $EndComp
 $Comp
-L 74xx:74LS76 U24
+L 74xx:74LS76 U42
 U 3 1 5F867596
 P 2000 6950
-F 0 "U24" V 1850 6850 50  0000 L CNN
+F 0 "U42" V 1850 6850 50  0000 L CNN
 F 1 "74LS76" V 2150 6800 50  0000 L CNN
 F 2 "" H 2000 6950 50  0001 C CNN
@@
 	9150 1500 9000 1500
 $Comp
-L power:VCC #PWR076
+L power:VCC #PWR0125
 U 1 1 5F8FA7AA
 P 9900 1000
-F 0 "#PWR076" H 9900 850 50  0001 C CNN
+F 0 "#PWR0125" H 9900 850 50  0001 C CNN
 F 1 "VCC" H 9917 1173 50  0000 C CNN
 F 2 "" H 9900 1000 50  0001 C CNN
@@
 $EndComp
 $Comp
-L power:VCC #PWR077
+L power:VCC #PWR0126
 U 1 1 5F8FB2DB
 P 9900 1800
-F 0 "#PWR077" H 9900 1650 50  0001 C CNN
+F 0 "#PWR0126" H 9900 1650 50  0001 C CNN
 F 1 "VCC" H 9917 1973 50  0000 C CNN
 F 2 "" H 9900 1800 50  0001 C CNN
@@
 $EndComp
 $Comp
-L power:VCC #PWR072
+L power:VCC #PWR0121
 U 1 1 5FA36B87
 P 6800 950
-F 0 "#PWR072" H 6800 800 50  0001 C CNN
+F 0 "#PWR0121" H 6800 800 50  0001 C CNN
 F 1 "VCC" H 6817 1123 50  0000 C CNN
 F 2 "" H 6800 950 50  0001 C CNN
@@
 $EndComp
 $Comp
-L power:VCC #PWR071
+L power:VCC #PWR0120
 U 1 1 5FA38CD9
 P 6300 1550
-F 0 "#PWR071" H 6300 1400 50  0001 C CNN
+F 0 "#PWR0120" H 6300 1400 50  0001 C CNN
 F 1 "VCC" H 6300 1700 50  0000 C CNN
 F 2 "" H 6300 1550 50  0001 C CNN
@@
 $EndComp
 $Comp
-L Device:C C7
+L Device:C C8
 U 1 1 5FA3AAEC
 P 6000 1500
-F 0 "C7" H 6050 1600 50  0000 L CNN
+F 0 "C8" H 6050 1600 50  0000 L CNN
 F 1 "10n" H 6050 1400 50  0000 L CNN
 F 2 "" H 6038 1350 50  0001 C CNN
@@
 $EndComp
 $Comp
-L Device:C C6
+L Device:C C7
 U 1 1 5FA3C597
 P 5700 1500
-F 0 "C6" H 5750 1600 50  0000 L CNN
+F 0 "C7" H 5750 1600 50  0000 L CNN
 F 1 "10n" H 5750 1400 50  0000 L CNN
 F 2 "" H 5738 1350 50  0001 C CNN
@@
 Connection ~ 5700 1150
 $Comp
-L Device:R R9
+L Device:R R12
 U 1 1 5FA70B5D
 P 7650 1550
-F 0 "R9" V 7550 1550 50  0000 C CNN
+F 0 "R12" V 7550 1550 50  0000 C CNN
 F 1 "100K" V 7750 1550 50  0000 C CNN
 F 2 "" V 7580 1550 50  0001 C CNN
@@
 $EndComp
 $Comp
-L Device:R R10
+L Device:R R13
 U 1 1 5FA7C626
 P 8050 1550
-F 0 "R10" V 7950 1550 50  0000 C CNN
+F 0 "R13" V 7950 1550 50  0000 C CNN
 F 1 "1K" V 8150 1550 50  0000 C CNN
 F 2 "" V 7980 1550 50  0001 C CNN
@@
 	8200 1550 8300 1550
 $Comp
-L power:VCC #PWR074
+L power:VCC #PWR0123
 U 1 1 5FAAF97C
 P 8300 1550
-F 0 "#PWR074" H 8300 1400 50  0001 C CNN
+F 0 "#PWR0123" H 8300 1400 50  0001 C CNN
 F 1 "VCC" H 8317 1723 50  0000 C CNN
 F 2 "" H 8300 1550 50  0001 C CNN
@@
 DCLK
 $Comp
-L 74xx:74LS08 U22
+L 74xx:74LS08 U33
 U 5 1 5FBA25F0
 P 2600 6950
-F 0 "U22" V 2450 6900 50  0000 L CNN
+F 0 "U33" V 2450 6900 50  0000 L CNN
 F 1 "74LS08" V 2750 6800 50  0000 L CNN
 F 2 "" H 2600 6950 50  0001 C CNN
@@
 $EndComp
 $Comp
-L 74xx:74LS273 U25
+L 74xx:74LS273 U43
 U 1 1 5FBCA7B4
 P 2600 1650
-F 0 "U25" H 2350 2300 50  0000 C CNN
+F 0 "U43" H 2350 2300 50  0000 C CNN
 F 1 "74LS273" H 2800 1000 50  0000 C CNN
 F 2 "" H 2600 1650 50  0001 C CNN
@@
 	1650 2050 2100 2050
 $Comp
-L 74xx:74LS08 U22
+L 74xx:74LS08 U33
 U 1 1 5FBA0032
 P 1350 2050
-F 0 "U22" H 1300 2250 50  0000 C CNN
+F 0 "U33" H 1300 2250 50  0000 C CNN
 F 1 "74LS08" H 1350 1850 50  0000 C CNN
 F 2 "" H 1350 2050 50  0001 C CNN
@@
 CLK
 $Comp
-L power:VCC #PWR064
+L power:VCC #PWR0113
 U 1 1 5FC72686
 P 2600 850
-F 0 "#PWR064" H 2600 700 50  0001 C CNN
+F 0 "#PWR0113" H 2600 700 50  0001 C CNN
 F 1 "VCC" H 2617 1023 50  0000 C CNN
 F 2 "" H 2600 850 50  0001 C CNN
@@
 $EndComp
 $Comp
-L power:GND #PWR065
+L power:GND #PWR0114
 U 1 1 5FC72DA1
 P 2600 2450
-F 0 "#PWR065" H 2600 2200 50  0001 C CNN
+F 0 "#PWR0114" H 2600 2200 50  0001 C CNN
 F 1 "GND" H 2605 2277 50  0000 C CNN
 F 2 "" H 2600 2450 50  0001 C CNN
@@
 $EndComp
 $Comp
-L power:VCC #PWR066
+L power:VCC #PWR0115
 U 1 1 5FC923A3
 P 3350 2750
-F 0 "#PWR066" H 3350 2600 50  0001 C CNN
+F 0 "#PWR0115" H 3350 2600 50  0001 C CNN
 F 1 "VCC" H 3367 2923 50  0000 C CNN
 F 2 "" H 3350 2750 50  0001 C CNN
@@
 $EndComp
 $Comp
-L power:VCC #PWR062
+L power:VCC #PWR0111
 U 1 1 5FCB56E7
 P 1200 6450
-F 0 "#PWR062" H 1200 6300 50  0001 C CNN
+F 0 "#PWR0111" H 1200 6300 50  0001 C CNN
 F 1 "VCC" H 1217 6623 50  0000 C CNN
 F 2 "" H 1200 6450 50  0001 C CNN
@@
 	2000 6450 2600 6450
 $Comp
-L power:GND #PWR067
+L power:GND #PWR0116
 U 1 1 61DE4719
 P 3350 2950
-F 0 "#PWR067" H 3350 2700 50  0001 C CNN
+F 0 "#PWR0116" H 3350 2700 50  0001 C CNN
 F 1 "GND" H 3355 2777 50  0000 C CNN
 F 2 "" H 3350 2950 50  0001 C CNN
@@
 Connection ~ 3350 2950
 $Comp
-L power:GND #PWR070
+L power:GND #PWR0119
 U 1 1 61DE57F8
 P 5850 1750
-F 0 "#PWR070" H 5850 1500 50  0001 C CNN
+F 0 "#PWR0119" H 5850 1500 50  0001 C CNN
 F 1 "GND" H 5855 1577 50  0000 C CNN
 F 2 "" H 5850 1750 50  0001 C CNN
@@
 $EndComp
 $Comp
-L power:GND #PWR073
+L power:GND #PWR0122
 U 1 1 61DE6334
 P 6800 1750
-F 0 "#PWR073" H 6800 1500 50  0001 C CNN
+F 0 "#PWR0122" H 6800 1500 50  0001 C CNN
 F 1 "GND" H 6805 1577 50  0000 C CNN
 F 2 "" H 6800 1750 50  0001 C CNN
@@
 $EndComp
 $Comp
-L power:GND #PWR075
+L power:GND #PWR0124
 U 1 1 61DE7F30
 P 9200 2750
-F 0 "#PWR075" H 9200 2500 50  0001 C CNN
+F 0 "#PWR0124" H 9200 2500 50  0001 C CNN
 F 1 "GND" H 9205 2577 50  0000 C CNN
 F 2 "" H 9200 2750 50  0001 C CNN
@@
 $EndComp
 $Comp
-L power:GND #PWR063
+L power:GND #PWR0112
 U 1 1 61DEAD62
 P 1200 7450
-F 0 "#PWR063" H 1200 7200 50  0001 C CNN
+F 0 "#PWR0112" H 1200 7200 50  0001 C CNN
 F 1 "GND" H 1205 7277 50  0000 C CNN
 F 2 "" H 1200 7450 50  0001 C CNN
@@
 $EndComp
 $Comp
-L sap-be:28C16 U?
+L sap:28C16 U?
 U 1 1 62226BB7
 P 4050 2050
 AR Path="/62226BB7" Ref="U?"  Part="1"
-AR Path="/591ACD24/62226BB7" Ref="U26"  Part="1"
-F 0 "U26" H 3750 3050 50  0000 C CNN
+AR Path="/591ACD24/62226BB7" Ref="U44"  Part="1"
+F 0 "U44" H 3750 3050 50  0000 C CNN
 F 1 "28C16" H 4300 1050 50  0000 C CNN
 F 2 "" H 4050 2050 50  0000 C CNN
@@
 	1    0    0    -1
 $EndComp
-Wire Bus Line
-	1700 950  1700 1750
-$Comp
-L power:VCC #PWR068
+$Comp
+L power:VCC #PWR0117
 U 1 1 62353D74
 P 4050 1000
-F 0 "#PWR068" H 4050 850 50  0001 C CNN
+F 0 "#PWR0117" H 4050 850 50  0001 C CNN
 F 1 "VCC" H 4067 1173 50  0000 C CNN
 F 2 "" H 4050 1000 50  0001 C CNN
@@
 $EndComp
 $Comp
-L power:GND #PWR069
+L power:GND #PWR0118
 U 1 1 62354C0E
 P 4050 3100
-F 0 "#PWR069" H 4050 2850 50  0001 C CNN
+F 0 "#PWR0118" H 4050 2850 50  0001 C CNN
 F 1 "GND" H 4055 2927 50  0000 C CNN
 F 2 "" H 4050 3100 50  0001 C CNN
@@
 	1    0    0    -1
 $EndComp
+Wire Bus Line
+	1700 950  1700 1750
 $EndSCHEMATC
