File: kicad/output.sch (KiCad schematic (older format))
At the start: 14 parts, among them U22 74HC74, U23 74LS273, U24 28C16, U25 74LS76, U26 74LS139, U27 NE555

Commit message: Update bugfix version to use updated kicad libraries
Parts:
- removed AFF1, AFF2, AFF3, AFF4: LTS-6980HR, Displays_7-Segment:7SegmentLED_LTS6760_LTS6780, symbol LTS-6980HR
- removed C6, C7: 10n, Capacitors_THT:C_Disc_D6_P5, symbol C
- removed R10: 100K, Resistors_THT:Resistor_Horizontal_RM7mm, symbol R
- removed R9: 1K, Resistors_THT:Resistor_Horizontal_RM7mm, symbol R
- removed U22: 74HC74, symbol 74HC74
- removed U23: 74LS273, Housings_DIP:DIP-20_W7.62mm_LongPads, symbol 74LS273
- removed U24: 28C16, Housings_DIP:DIP-24_W15.24mm_LongPads, symbol 28C16
- removed U25: 74LS76, Housings_DIP:DIP-16_W7.62mm_LongPads, symbol 74LS76
- removed U26: 74LS139, Housings_DIP:DIP-16_W7.62mm_LongPads, symbol 74LS139
- removed U27: NE555, Housings_DIP:DIP-8_W7.62mm_LongPads, symbol NE555
- added AFF1, AFF2, AFF3, AFF4: LTS-6980HR, Display_7Segment:7SegmentLED_LTS6760_LTS6780, symbol Display_Character:LTS-6980HR
- added C6, C7: 10n, symbol Device:C
- added R10: 1K, symbol Device:R
- added R9: 100K, symbol Device:R
- added U23: 74LS139, symbol 74xx:74LS139
- added U24: 74LS76, symbol 74xx:74LS76
- added U26: 28C16, symbol sap-be:28C16
- added U27: LM555, symbol Timer:LM555
- added U?: 74LS377, symbol 74xx:74LS377
Connections:
- net labels added: ~LOAD
- net labels removed: LOAD, OCLK, ~CLR
- wire segments 120 -> 139
- no-connect marks 3 -> 2

Commit message: update kicad project name
Parts:
- U26: symbol sap-be:28C16 -> sap:28C16
Changed lines of the file:
@@
 $EndComp
 $Comp
-L sap-be:28C16 U?
+L sap:28C16 U?
 U 1 1 62226BB7
 P 4050 2050
