File: kicad/programcounter.sch (KiCad schematic (older format))
At the start: 6 parts, among them U13 74LS161, U14 74LS245

Commit message: bugfixed design
Parts:
- renumbered U13 to U20, U14 to U21
Changed lines of the file:
@@
 LIBS:valves
 LIBS:switches
-LIBS:74xxx
-LIBS:28c16
 LIBS:sap-be-cache
-EELAYER 24 0
+EELAYER 25 0
 EELAYER END
 $Descr A4 11693 8268
@@
 ~LOAD
 $Comp
-L 74LS161 U13
+L 74LS161 U20
 U 1 1 591B044D
 P 5450 2600
-F 0 "U13" H 5500 2700 50  0000 C CNN
+F 0 "U20" H 5500 2700 50  0000 C CNN
 F 1 "74LS161" H 5550 2400 50  0000 C CNN
 F 2 "Housings_DIP:DIP-16_W7.62mm_LongPads" H 5450 2600 50  0001 C CNN
@@
 $EndComp
 $Comp
-L 74LS245 U14
+L 74LS245 U21
 U 1 1 591B0585
 P 5450 4050
-F 0 "U14" H 5550 4625 50  0000 L BNN
+F 0 "U21" H 5550 4625 50  0000 L BNN
 F 1 "74LS245" H 5500 3475 50  0000 L TNN
 F 2 "Housings_DIP:DIP-20_W7.62mm_LongPads" H 5450 4050 50  0001 C CNN
@@
 r3
 $Comp
-L GND #PWR029
+L GND #PWR28
 U 1 1 591B1C69
 P 6150 3200
-F 0 "#PWR029" H 6150 2950 50  0001 C CNN
+F 0 "#PWR28" H 6150 2950 50  0001 C CNN
 F 1 "GND" H 6150 3050 50  0000 C CNN
 F 2 "" H 6150 3200 50  0000 C CNN
@@
 r3
 $Comp
-L GND #PWR030
+L GND #PWR29
 U 1 1 591B25A3
 P 7800 4100
-F 0 "#PWR030" H 7800 3850 50  0001 C CNN
+F 0 "#PWR29" H 7800 3850 50  0001 C CNN
 F 1 "GND" H 7800 3950 50  0000 C CNN
 F 2 "" H 7800 4100 50  0000 C CNN
@@
 	4250 1700 3700 1700
 $Comp
-L GND #PWR031
+L GND #PWR27
 U 1 1 59145790
 P 4250 4450
-F 0 "#PWR031" H 4250 4200 50  0001 C CNN
+F 0 "#PWR27" H 4250 4200 50  0001 C CNN
 F 1 "GND" H 4250 4300 50  0000 C CNN
 F 2 "" H 4250 4450 50  0000 C CNN

Commit message: design as built
Parts:
- renumbered D18 to D801, D19 to D802, D20 to D803, D21 to D804, U20 to U801, U21 to U802
Changed lines of the file:
@@
 LIBS:valves
 LIBS:switches
+LIBS:74xxx
+LIBS:28c16
+LIBS:ne556
 LIBS:sap-be-cache
 EELAYER 25 0
@@
 Sheet 6 12
 Title "Simple As Possible computer by Ben Eater"
-Date "2017-05-10"
-Rev "1"
+Date "2018-06-03"
+Rev "2"
 Comp "Schematic released as CC BY-SA"
 Comment1 "Schematic capture by Vincent Sanders"
@@
 ~LOAD
 $Comp
-L 74LS161 U20
+L 74LS161 U801
 U 1 1 591B044D
 P 5450 2600
-F 0 "U20" H 5500 2700 50  0000 C CNN
+F 0 "U801" H 5500 2700 50  0000 C CNN
 F 1 "74LS161" H 5550 2400 50  0000 C CNN
 F 2 "Housings_DIP:DIP-16_W7.62mm_LongPads" H 5450 2600 50  0001 C CNN
@@
 $EndComp
 $Comp
-L 74LS245 U21
+L 74LS245 U802
 U 1 1 591B0585
 P 5450 4050
-F 0 "U21" H 5550 4625 50  0000 L BNN
+F 0 "U802" H 5550 4625 50  0000 L BNN
 F 1 "74LS245" H 5500 3475 50  0000 L TNN
 F 2 "Housings_DIP:DIP-20_W7.62mm_LongPads" H 5450 4050 50  0001 C CNN
@@
 r3
 $Comp
-L GND #PWR28
+L GND #PWR038
 U 1 1 591B1C69
 P 6150 3200
-F 0 "#PWR28" H 6150 2950 50  0001 C CNN
+F 0 "#PWR038" H 6150 2950 50  0001 C CNN
 F 1 "GND" H 6150 3050 50  0000 C CNN
 F 2 "" H 6150 3200 50  0000 C CNN
@@
 r[0..7]
 $Comp
-L LED D18
+L LED D801
 U 1 1 591B255B
 P 6600 3750
-F 0 "D18" H 6600 3850 50  0000 C CNN
+F 0 "D801" H 6600 3850 50  0000 C CNN
 F 1 "LED" H 6600 3650 50  0000 C CNN
 F 2 "LEDs:LED-5MM" H 6600 3750 50  0001 C CNN
@@
 $EndComp
 $Comp
-L LED D19
+L LED D802
 U 1 1 591B2562
 P 6900 3750
-F 0 "D19" H 6900 3850 50  0000 C CNN
+F 0 "D802" H 6900 3850 50  0000 C CNN
 F 1 "LED" H 6900 3650 50  0000 C CNN
 F 2 "LEDs:LED-5MM" H 6900 3750 50  0001 C CNN
@@
 $EndComp
 $Comp
-L LED D20
+L LED D803
 U 1 1 591B2569
 P 7200 3750
-F 0 "D20" H 7200 3850 50  0000 C CNN
+F 0 "D803" H 7200 3850 50  0000 C CNN
 F 1 "LED" H 7200 3650 50  0000 C CNN
 F 2 "LEDs:LED-5MM" H 7200 3750 50  0001 C CNN
@@
 $EndComp
 $Comp
-L LED D21
+L LED D804
 U 1 1 591B2570
 P 7500 3750
-F 0 "D21" H 7500 3850 50  0000 C CNN
+F 0 "D804" H 7500 3850 50  0000 C CNN
 F 1 "LED" H 7500 3650 50  0000 C CNN
 F 2 "LEDs:LED-5MM" H 7500 3750 50  0001 C CNN
@@
 r3
 $Comp
-L GND #PWR29
+L GND #PWR039
 U 1 1 591B25A3
 P 7800 4100
-F 0 "#PWR29" H 7800 3850 50  0001 C CNN
+F 0 "#PWR039" H 7800 3850 50  0001 C CNN
 F 1 "GND" H 7800 3950 50  0000 C CNN
 F 2 "" H 7800 4100 50  0000 C CNN
@@
 	4250 1700 3700 1700
 $Comp
-L GND #PWR27
+L GND #PWR040
 U 1 1 59145790
 P 4250 4450
-F 0 "#PWR27" H 4250 4200 50  0001 C CNN
+F 0 "#PWR040" H 4250 4200 50  0001 C CNN
 F 1 "GND" H 4250 4300 50  0000 C CNN
 F 2 "" H 4250 4450 50  0000 C CNN

Commit message: Update to current kicad version
Parts:
- removed D801, D802, D803, D804: LED, LEDs:LED-5MM, symbol LED
- removed U801: 74LS161, Housings_DIP:DIP-16_W7.62mm_LongPads, symbol 74LS161
- removed U802: 74LS245, Housings_DIP:DIP-20_W7.62mm_LongPads, symbol 74LS245
- added BAR6: HDSP-4830_2, Display:HDSP-4830, symbol LED:HDSP-4830_2
- added RN8: 1K, Resistor_THT:R_Array_SIP9, symbol Device:R_Network08
- added U26: 74LS245, symbol 74xx:74LS245
- added U27: 74LS161, symbol 74xx:74LS161
Connections:
- net labels added: VCC, pc0, pc1, pc2, pc3, pc4, pc5, pc6, pc7, pc[0..7]
- net labels removed: r0, r1, r2, r3, r4, r5, r6, r7, r[0..7]
- wire segments 52 -> 54
- no-connect marks 1 -> 5
