File: kicad/ALU.sch (KiCad schematic (older format))
At the start: 7 parts, among them U1 74LS86, U2 74LS86, U3 74LS283, U4 74LS283, U46 7402, U47 74LS08, U5 74LS245

Commit message: Update to current kicad libraries
Parts:
- removed U1, U2: 74LS86, Housings_DIP:DIP-14_W7.62mm_LongPads, symbol 74LS86
- removed U3, U4: 74LS283, Housings_DIP:DIP-16_W7.62mm_LongPads, symbol 74LS283
- removed U46: 7402, symbol 7402
- removed U47: 74LS08, symbol 74LS08
- removed U5: 74LS245, Housings_DIP:DIP-20_W7.62mm_LongPads, symbol 74LS245
- added U1, U2: 74LS86, symbol 74xx:74LS86
- added U3: 74LS02, symbol 74xx:74LS02
- added U4: 74LS08, symbol 74xx:74LS08
- added U5, U6: 74LS283, symbol 74xx:74LS283
- added U7: 74LS245, symbol 74xx:74LS245
Connections:
- net labels added: GND, ra[0..7], rb[0..7]
- wire segments 120 -> 126

Commit message: update bus names and improve sheet text
Parts:
- added U33: 74LS08, symbol 74xx:74LS08
- renumbered U1 to U28, U2 to U29, U3 to U30, U5 to U31, U6 to U32, U7 to U34, U4 to U8
Changed lines of the file:
@@
 $Descr A4 11693 8268
 encoding utf-8
-Sheet 2 13
-Title "Simple As Possible computer by Ben Eater"
+Sheet 8 13
+Title "Simple As Possible computer"
 Date "2017-05-10"
 Rev "1"
 Comp "Schematic released as CC BY-SA"
-Comment1 "Schematic capture by Vincent Sanders"
+Comment1 "Schematic capture by Vincent Sanders of a design by Ben Eater"
 Comment2 "Arithmetic Logic Unit"
 Comment3 ""
@@
 	1500 2150 1500 2650
 $Comp
-L 74xx:74LS02 U3
+L 74xx:74LS02 U30
 U 1 1 5EDA51E2
 P 8300 4450
-F 0 "U3" H 8300 4450 50  0000 C CNN
+F 0 "U30" H 8300 4450 50  0000 C CNN
 F 1 "74LS02" H 8550 4350 50  0000 C CNN
 F 2 "" H 8300 4450 50  0001 C CNN
@@
 $EndComp
 $Comp
-L 74xx:74LS02 U3
+L 74xx:74LS02 U30
 U 2 1 5EDA6FFD
 P 8300 4850
-F 0 "U3" H 8300 4850 50  0000 C CNN
+F 0 "U30" H 8300 4850 50  0000 C CNN
 F 1 "74LS02" H 8550 4750 50  0000 C CNN
 F 2 "" H 8300 4850 50  0001 C CNN
@@
 $EndComp
 $Comp
-L 74xx:74LS02 U3
+L 74xx:74LS02 U30
 U 3 1 5EDA7B2C
 P 8300 5250
-F 0 "U3" H 8300 5250 50  0000 C CNN
+F 0 "U30" H 8300 5250 50  0000 C CNN
 F 1 "74LS02" H 8550 5150 50  0000 C CNN
 F 2 "" H 8300 5250 50  0001 C CNN
@@
 $EndComp
 $Comp
-L 74xx:74LS02 U3
+L 74xx:74LS02 U30
 U 4 1 5EDA92E1
 P 8300 5650
-F 0 "U3" H 8300 5650 50  0000 C CNN
+F 0 "U30" H 8300 5650 50  0000 C CNN
 F 1 "74LS02" H 8550 5550 50  0000 C CNN
 F 2 "" H 8300 5650 50  0001 C CNN
@@
 $EndComp
 $Comp
-L 74xx:74LS02 U3
+L 74xx:74LS02 U30
 U 5 1 5EDAE91C
 P 2400 6950
-F 0 "U3" V 2250 6900 50  0000 L CNN
+F 0 "U30" V 2250 6900 50  0000 L CNN
 F 1 "74LS02" V 2550 6800 50  0000 L CNN
 F 2 "" H 2400 6950 50  0001 C CNN
@@
 $EndComp
 $Comp
-L 74xx:74LS08 U4
+L 74xx:74LS08 U8
 U 1 1 5EDFEA86
 P 9200 4650
-F 0 "U4" H 9200 4850 50  0000 C CNN
+F 0 "U8" H 9200 4850 50  0000 C CNN
 F 1 "74LS08" H 9200 4450 50  0000 C CNN
 F 2 "" H 9200 4650 50  0001 C CNN
@@
 $EndComp
 $Comp
-L 74xx:74LS08 U4
+L 74xx:74LS08 U8
 U 2 1 5EE00151
 P 9200 5450
-F 0 "U4" H 9200 5650 50  0000 C CNN
+F 0 "U8" H 9200 5650 50  0000 C CNN
 F 1 "74LS08" H 9200 5250 50  0000 C CNN
 F 2 "" H 9200 5450 50  0001 C CNN
@@
 $EndComp
 $Comp
-L 74xx:74LS08 U4
+L 74xx:74LS08 U8
 U 3 1 5EE01C3C
 P 10100 5050
-F 0 "U4" H 10100 5250 50  0000 C CNN
+F 0 "U8" H 10100 5250 50  0000 C CNN
 F 1 "74LS08" H 10100 4850 50  0000 C CNN
 F 2 "" H 10100 5050 50  0001 C CNN
@@
 $EndComp
 $Comp
-L 74xx:74LS08 U4
+L 74xx:74LS08 U8
 U 5 1 5EE04A56
 P 3050 6950
-F 0 "U4" V 2900 6900 50  0000 L CNN
+F 0 "U8" V 2900 6900 50  0000 L CNN
 F 1 "74LS08" V 3200 6800 50  0000 L CNN
 F 2 "" H 3050 6950 50  0001 C CNN
@@
 	7400 4050 7400 6000
 $Comp
-L 74xx:74LS86 U1
+L 74xx:74LS86 U28
 U 1 1 5EEF4E86
 P 2300 2250
-F 0 "U1" H 2300 2450 50  0000 C CNN
+F 0 "U28" H 2300 2450 50  0000 C CNN
 F 1 "74LS86" H 2300 2050 50  0000 C CNN
 F 2 "" H 2300 2250 50  0001 C CNN
@@
 $EndComp
 $Comp
-L 74xx:74LS86 U1
+L 74xx:74LS86 U28
 U 2 1 5EEF6113
 P 2300 2750
-F 0 "U1" H 2300 2950 50  0000 C CNN
+F 0 "U28" H 2300 2950 50  0000 C CNN
 F 1 "74LS86" H 2300 2550 50  0000 C CNN
 F 2 "" H 2300 2750 50  0001 C CNN
@@
 $EndComp
 $Comp
-L 74xx:74LS86 U1
+L 74xx:74LS86 U28
 U 3 1 5EEFA088
 P 2300 3300
-F 0 "U1" H 2300 3500 50  0000 C CNN
+F 0 "U28" H 2300 3500 50  0000 C CNN
 F 1 "74LS86" H 2300 3100 50  0000 C CNN
 F 2 "" H 2300 3300 50  0001 C CNN
@@
 $EndComp
 $Comp
-L 74xx:74LS86 U1
+L 74xx:74LS86 U28
 U 4 1 5EEFAF03
 P 2300 3800
-F 0 "U1" H 2300 4000 50  0000 C CNN
+F 0 "U28" H 2300 4000 50  0000 C CNN
 F 1 "74LS86" H 2300 3600 50  0000 C CNN
 F 2 "" H 2300 3800 50  0001 C CNN
@@
 $EndComp
 $Comp
-L 74xx:74LS86 U1
+L 74xx:74LS86 U28
 U 5 1 5EEFC1D0
 P 1100 6950
-F 0 "U1" V 950 6900 50  0000 L CNN
+F 0 "U28" V 950 6900 50  0000 L CNN
 F 1 "74LS86" V 1250 6800 50  0000 L CNN
 F 2 "" H 1100 6950 50  0001 C CNN
@@
 $EndComp
 $Comp
-L 74xx:74LS86 U2
+L 74xx:74LS86 U29
 U 5 1 5EF0B90C
 P 1750 6950
-F 0 "U2" V 1600 6900 50  0000 L CNN
+F 0 "U29" V 1600 6900 50  0000 L CNN
 F 1 "74LS86" V 1900 6800 50  0000 L CNN
 F 2 "" H 1750 6950 50  0001 C CNN
@@
 $EndComp
 $Comp
-L 74xx:74LS86 U2
+L 74xx:74LS86 U29
 U 1 1 5EF0C990
 P 2300 4300
-F 0 "U2" H 2300 4500 50  0000 C CNN
+F 0 "U29" H 2300 4500 50  0000 C CNN
 F 1 "74LS86" H 2300 4100 50  0000 C CNN
 F 2 "" H 2300 4300 50  0001 C CNN
@@
 $EndComp
 $Comp
-L 74xx:74LS86 U2
+L 74xx:74LS86 U29
 U 2 1 5EF0DCF1
 P 2300 4750
-F 0 "U2" H 2300 4950 50  0000 C CNN
+F 0 "U29" H 2300 4950 50  0000 C CNN
 F 1 "74LS86" H 2300 4550 50  0000 C CNN
 F 2 "" H 2300 4750 50  0001 C CNN
@@
 $EndComp
 $Comp
-L 74xx:74LS86 U2
+L 74xx:74LS86 U29
 U 3 1 5EF0F0BC
 P 2300 5250
-F 0 "U2" H 2300 5450 50  0000 C CNN
+F 0 "U29" H 2300 5450 50  0000 C CNN
 F 1 "74LS86" H 2300 5050 50  0000 C CNN
 F 2 "" H 2300 5250 50  0001 C CNN
@@
 $EndComp
 $Comp
-L 74xx:74LS86 U2
+L 74xx:74LS86 U29
 U 4 1 5EF10479
 P 2300 5750
-F 0 "U2" H 2300 5950 50  0000 C CNN
+F 0 "U29" H 2300 5950 50  0000 C CNN
 F 1 "74LS86" H 2300 5550 50  0000 C CNN
 F 2 "" H 2300 5750 50  0001 C CNN
@@
 	1200 1550 3100 1550
 $Comp
-L 74xx:74LS283 U6
+L 74xx:74LS283 U32
 U 1 1 5F085B2E
 P 4000 4750
-F 0 "U6" H 3750 5400 50  0000 C CNN
+F 0 "U32" H 3750 5400 50  0000 C CNN
 F 1 "74LS283" H 3800 4100 50  0000 C CNN
 F 2 "" H 4000 4750 50  0001 C CNN
@@
 	3300 4450 3500 4450
 $Comp
-L power:GND #PWR010
+L power:GND #PWR086
 U 1 1 5F24608C
 P 4000 5550
-F 0 "#PWR010" H 4000 5300 50  0001 C CNN
+F 0 "#PWR086" H 4000 5300 50  0001 C CNN
 F 1 "GND" H 4005 5377 50  0000 C CNN
 F 2 "" H 4000 5550 50  0001 C CNN
@@
 $EndComp
 $Comp
-L 74xx:74LS283 U5
+L 74xx:74LS283 U31
 U 1 1 5F25DC09
 P 4000 2450
-F 0 "U5" H 3750 3100 50  0000 C CNN
+F 0 "U31" H 3750 3100 50  0000 C CNN
 F 1 "74LS283" H 3800 1800 50  0000 C CNN
 F 2 "" H 4000 2450 50  0001 C CNN
@@
 	3300 2450 3500 2450
 $Comp
-L power:GND #PWR08
+L power:GND #PWR084
 U 1 1 5F2C1503
 P 4000 3250
-F 0 "#PWR08" H 4000 3000 50  0001 C CNN
+F 0 "#PWR084" H 4000 3000 50  0001 C CNN
 F 1 "GND" H 4005 3077 50  0000 C CNN
 F 2 "" H 4000 3250 50  0001 C CNN
@@
 	2600 2750 3500 2750
 $Comp
-L 74xx:74LS245 U7
+L 74xx:74LS245 U34
 U 1 1 5F32FA27
 P 6100 2450
-F 0 "U7" H 5850 3100 50  0000 C CNN
+F 0 "U34" H 5850 3100 50  0000 C CNN
 F 1 "74LS245" H 5900 1800 50  0000 C CNN
 F 2 "" H 6100 2450 50  0001 C CNN
@@
 	4600 2450 4600 3600
 $Comp
-L power:GND #PWR013
+L power:GND #PWR089
 U 1 1 5F476FC1
 P 6100 3250
-F 0 "#PWR013" H 6100 3000 50  0001 C CNN
+F 0 "#PWR089" H 6100 3000 50  0001 C CNN
 F 1 "GND" H 6105 3077 50  0000 C CNN
 F 2 "" H 6100 3250 50  0001 C CNN
@@
 $EndComp
 $Comp
-L power:GND #PWR06
+L power:GND #PWR082
 U 1 1 5F511F35
 P 900 7450
-F 0 "#PWR06" H 900 7200 50  0001 C CNN
+F 0 "#PWR082" H 900 7200 50  0001 C CNN
 F 1 "GND" H 905 7277 50  0000 C CNN
 F 2 "" H 900 7450 50  0001 C CNN
@@
 	2600 5250 2900 5250
 $Comp
-L power:VCC #PWR011
+L power:VCC #PWR087
 U 1 1 61E0DBC7
 P 5500 2850
-F 0 "#PWR011" H 5500 2700 50  0001 C CNN
+F 0 "#PWR087" H 5500 2700 50  0001 C CNN
 F 1 "VCC" H 5500 3000 50  0000 C CNN
 F 2 "" H 5500 2850 50  0001 C CNN
@@
 $EndComp
 $Comp
-L power:VCC #PWR012
+L power:VCC #PWR088
 U 1 1 61E0E043
 P 6100 1650
-F 0 "#PWR012" H 6100 1500 50  0001 C CNN
+F 0 "#PWR088" H 6100 1500 50  0001 C CNN
 F 1 "VCC" H 6100 1800 50  0000 C CNN
 F 2 "" H 6100 1650 50  0001 C CNN
@@
 $EndComp
 $Comp
-L power:VCC #PWR09
+L power:VCC #PWR085
 U 1 1 61E10B94
 P 4000 3950
-F 0 "#PWR09" H 4000 3800 50  0001 C CNN
+F 0 "#PWR085" H 4000 3800 50  0001 C CNN
 F 1 "VCC" H 4000 4100 50  0000 C CNN
 F 2 "" H 4000 3950 50  0001 C CNN
@@
 $EndComp
 $Comp
-L power:VCC #PWR07
+L power:VCC #PWR083
 U 1 1 61E12AF2
 P 4000 1650
-F 0 "#PWR07" H 4000 1500 50  0001 C CNN
+F 0 "#PWR083" H 4000 1500 50  0001 C CNN
 F 1 "VCC" H 4000 1800 50  0000 C CNN
 F 2 "" H 4000 1650 50  0001 C CNN
@@
 $EndComp
 $Comp
-L power:VCC #PWR05
+L power:VCC #PWR081
 U 1 1 61E19004
 P 900 6450
-F 0 "#PWR05" H 900 6300 50  0001 C CNN
+F 0 "#PWR081" H 900 6300 50  0001 C CNN
 F 1 "VCC" H 900 6600 50  0000 C CNN
 F 2 "" H 900 6450 50  0001 C CNN
@@
 Wire Bus Line
 	7150 1450 7150 2750
+$Comp
+L 74xx:74LS08 U33
+U 4 1 5EAC53BC
+P 6050 7000
+F 0 "U33" H 6050 7200 50  0000 C CNN
+F 1 "74LS08" H 6050 6800 50  0000 C CNN
+F 2 "" H 6050 7000 50  0001 C CNN
+F 3 "http://www.ti.com/lit/gpn/sn74LS08" H 6050 7000 50  0001 C CNN
+	4    6050 7000
+	1    0    0    -1
+$EndComp
 $EndSCHEMATC
